File: New_Atmega 2560/New_Atmega 2560.kicad_pcb (KiCad board)
At the start: 2 copper layers, 12 parts, among them J1 Barrel_Jack_Switch, U1 ATmega2560-16A

Commit message: Add files via upload
Parts:
- added C16: 100n, Capacitor_SMD:C_0603_1608Metric, F.Cu at (123.5, 98.7)
- added J2: Conn_01x08, Connector_PinHeader_2.54mm:PinHeader_2x18_P2.54mm_Vertical, F.Cu at (100.1, 76.4)
- C1, C7: value 100n -> ~
- C3, C4: value ~ -> 100n
- moved CPC1 51.6 mm to (123.5, 101.2)
- moved PC1 51.6 mm to (123.5, 103.8)
- moved C2 51.5 mm to (119.5, 96.2)
- moved C3 51.5 mm to (119.5, 98.7)
- moved C4 51.5 mm to (119.5, 101.2)
- moved C5 51.5 mm to (119.5, 103.8)
- moved C1 51.5 mm to (119.5, 93.7)
- moved C6 51.0 mm to (123.5, 93.7)
- moved C7 51.0 mm to (123.5, 96.2)
- moved U1 29.6 mm to (114.1, 83.3)
- moved D1 26.1 mm to (109.1, 112.3)
- moved J1 26.1 mm to (110.4, 94.8)
Connections:
- net Net-(U1-VCC-Pad10) renamed /VCC
- C1 pad 1: /AREF -> /XTAL2
- C2 pad 1: +5V -> /VIN
- C2 pad 2: Net-(C2-Pad2) -> GND
- C3 pad 1: /XTAL2 -> /AREF
- C4 pad 1: /XTAL1 -> +5V
- C5 pad 1: /VIN -> +5V
- C6 pad 2: Net-(C2-Pad2) -> GND
- C7 pad 1: +5V -> /XTAL1
- C7 pad 2: Net-(C2-Pad2) -> GND
- U1 pad 100: unconnected-(U1-AVCC-Pad100) -> /AVCC
- U1 pad 11: Net-(U1-GND-Pad11) -> GND
- U1 pad 30: unconnected-(U1-~{RESET}-Pad30) -> /RESET
- U1 pad 32: Net-(U1-GND-Pad11) -> GND
- U1 pad 62: Net-(U1-GND-Pad11) -> GND
- U1 pad 81: Net-(U1-GND-Pad11) -> GND
- U1 pad 99: Net-(U1-GND-Pad11) -> GND
Routing:
- net /VCC: track 15.0 -> 0.00 mm
- net Net-(U1-GND-Pad11): track 14.1 -> 0.00 mm
