File: New_Atmega 2560/New_Atmega 2560.kicad_pcb (KiCad board)
At the start: 2 copper layers, 14 parts, among them J1 Barrel_Jack_Switch, J2 Conn_01x08, U1 ATmega2560-16A

Commit message: PCB電路圖設計
Parts:
- added ADCH1: ADCH, Connector_PinHeader_2.54mm:PinHeader_1x08_P2.54mm_Vertical, F.Cu at (158.0, 75.3)
- added C10: 1u, Capacitor_SMD:C_0603_1608Metric, F.Cu at (157.7, 115.9)
- added C11: C, Capacitor_SMD:C_0603_1608Metric, F.Cu at (157.7, 118.4)
- added C12: 1uF, Capacitor_SMD:C_0603_1608Metric, F.Cu at (70.5, 47.5)
- added C13: 100nF, Capacitor_SMD:C_0603_1608Metric, F.Cu at (64.5, 52.8)
- added C14: C_US, Capacitor_SMD:C_0603_1608Metric, F.Cu at (67.0, 48.0)
- added C15: C_US, Capacitor_SMD:C_0603_1608Metric, F.Cu at (63.0, 48.0)
- added C17: C_US, Capacitor_SMD:C_0603_1608Metric, F.Cu at (68.5, 59.5)
- added C18: 100nF, Capacitor_SMD:C_0603_1608Metric_Pad1.08x0.95mm_HandSolder, F.Cu at (205.8, 95.1)
- added C8: 100n, Capacitor_SMD:C_0603_1608Metric, F.Cu at (157.7, 110.9)
- added C9: 100n, Capacitor_SMD:C_0603_1608Metric, F.Cu at (157.7, 113.4)
- added D2: CD1206-S01575, Diode_SMD:D_MiniMELF, F.Cu at (205.8, 102.8)
- added D3: CD1206-S01575, Diode_SMD:D_MiniMELF, F.Cu at (170.3, 119.6)
- added F1: MF-MSMF050, MF-MSMF050:FUSER_MF-MSMF050, F.Cu at (199.3, 103.6)
- added FB1: 30R 3A, mh2029-300y:L0805, F.Cu at (204.8, 106.0)
- added GREEN1: ON, LED_SMD:LED_PLCC_2835, F.Cu at (168.2, 90.0)
- added IC1: 1870_LD11117S50CTR, Package_TO_SOT_SMD:SOT-223-3_TabPin2, F.Cu at (182.0, 119.5)
- added IC2: MC33269D-5.0, Library:TO229P990X238-4N, F.Cu at (146.9, 62.3)
- added J2: Conn_01x08, Connector_PinHeader_2.54mm:PinHeader_2x02_P2.54mm_Vertical, F.Cu at (158.0, 97.7)
- added J3: Conn_01x08, Connector_PinHeader_2.54mm:PinHeader_2x02_P2.54mm_Vertical, F.Cu at (158.0, 104.8)
- added J4: Conn_01x08, Connector_PinHeader_2.54mm:PinHeader_2x02_P2.54mm_Vertical, F.Cu at (165.1, 97.7)
- added J5: Conn_01x08, Connector_PinHeader_2.54mm:PinHeader_2x02_P2.54mm_Vertical, F.Cu at (165.1, 104.8)
- added J6: Conn_01x10, Connector_PinHeader_2.54mm:PinHeader_2x02_P2.54mm_Vertical, F.Cu at (172.2, 97.7)
- added J7: Conn_01x06, Connector_PinHeader_2.54mm:PinHeader_2x02_P2.54mm_Vertical, F.Cu at (172.2, 104.8)
- added J8: Conn_PIC_ICSP_ICD, Connector_PinHeader_2.54mm:PinHeader_2x02_P2.54mm_Vertical, F.Cu at (181.4, 96.1)
- added J9: Conn_02x02_Counter_Clockwise, Connector_PinHeader_2.54mm:PinHeader_2x02_P2.54mm_Vertical, F.Cu at (181.4, 103.3)
- added P1: USB_C_Plug_USB2.0, Connector_USB:USB_C_Plug_Molex_105444, F.Cu at (191.1, 95.8)
- added R1: 1M, Resistor_SMD:R_0603_1608Metric, F.Cu at (157.7, 120.9)
- added R2: R, Resistor_SMD:R_0603_1608Metric, F.Cu at (84.2, 78.5)
- added R3: R, Resistor_SMD:R_0603_1608Metric, F.Cu at (88.2, 66.0)
- added R4: R, Resistor_SMD:R_0603_1608Metric, F.Cu at (88.2, 68.5)
- added R5: R, Resistor_SMD:R_0603_1608Metric, F.Cu at (88.2, 71.0)
- added R6: BRNCG0603MLC-05E, Resistor_SMD:R_0603_1608Metric, F.Cu at (88.2, 73.5)
- added R7: BRNCG0603MLC-05E, Resistor_SMD:R_0603_1608Metric, F.Cu at (88.2, 76.0)
- added RN1A1: 10k, Resistor_THT:R_Array_SIP8, F.Cu at (128.6, 75.1)
- added RN1B1: 10K, Resistor_THT:R_Array_SIP8, F.Cu at (128.6, 79.3)
- added RN1C1: 10K, Resistor_THT:R_Array_SIP8, F.Cu at (128.6, 83.4)
- added RN1D1: 10k, Resistor_THT:R_Array_SIP8, F.Cu at (128.6, 87.6)
- added RN2B1: 22R, Resistor_THT:R_Array_SIP8, F.Cu at (128.6, 91.8)
- added RN2C1: 22R, Resistor_THT:R_Array_SIP8, F.Cu at (128.6, 95.9)
- added RN3A1: 1K, Resistor_THT:R_Array_SIP8, F.Cu at (128.6, 100.1)
- added RN3B1: 1K, Resistor_THT:R_Array_SIP8, F.Cu at (128.6, 104.3)
- added RN3C1: 1k, Resistor_THT:R_Array_SIP8, F.Cu at (128.6, 108.4)
- added RN3D1: 1k, Resistor_THT:R_Array_SIP8, F.Cu at (181.2, 75.1)
- added RN4A1: 1k, Resistor_THT:R_Array_SIP8, F.Cu at (181.2, 79.3)
- added RN4B1: 1k, Resistor_THT:R_Array_SIP8, F.Cu at (181.2, 83.4)
- added RN4C1: 1k, Resistor_THT:R_Array_SIP8, F.Cu at (181.2, 87.6)
- added RN4C2: 1k, Resistor_THT:R_Array_SIP8, F.Cu at (181.2, 91.8)
- added RN5A1: 10K, Resistor_THT:R_Array_SIP8, F.Cu at (128.6, 112.6)
- added RN5C1: 10k, Resistor_THT:R_Array_SIP8, F.Cu at (128.6, 116.8)
- added RN5D1: 10k, Resistor_THT:R_Array_SIP8, F.Cu at (128.6, 121.0)
- added RX1: Yellow, LED_SMD:LED_PLCC_2835, F.Cu at (189.0, 100.5)
- added TX1: Yellow, LED_SMD:LED_PLCC_2835, F.Cu at (189.0, 104.8)
- added U2: LMV358IDGKR, Package_SO:MSOP-8_3x3mm_P0.65mm, F.Cu at (163.4, 112.0)
- added U3: LP2985-33DBVR, Package_TO_SOT_SMD:SOT-23-5, F.Cu at (162.8, 90.2)
- added U4: LMV358IDGKR, Package_SO:MSOP-8_3x3mm_P0.65mm, F.Cu at (163.4, 116.6)
- added U5: ATmega16U2-M, Package_DFN_QFN:QFN-32-1EP_5x5mm_P0.5mm_EP3.1x3.1mm, F.Cu at (70.0, 53.5)
- added XIO1: 18x2F-H8.5, Connector_PinHeader_2.54mm:PinHeader_2x18_P2.54mm_Vertical, F.Cu at (150.8, 75.3)
- added Y1: 16Hz, Crystal:Crystal_SMD_HC49-SD, F.Cu at (53.0, 43.0)
- added YELLOW1: L, LED_SMD:LED_0805_2012Metric, F.Cu at (173.2, 89.4)
- moved J1 111.0 mm to (27.5, 21.0), turned to -90 degrees
- moved J2 48.9 mm to (107.3, 28.0), turned to 90 degrees
- moved U1 39.8 mm to (89.5, 52.0)
Connections:
- J1 pad 2: unconnected-(J1-Pad2) -> GND
- U1 pad 1: unconnected-(U1-PG5-Pad1) -> /PG5
- U1 pad 12: unconnected-(U1-PH0-Pad12) -> /RXD2
- U1 pad 13: unconnected-(U1-PH1-Pad13) -> /TXD2
- U1 pad 15: unconnected-(U1-PH3-Pad15) -> /PH3
- U1 pad 16: unconnected-(U1-PH4-Pad16) -> /PH4
- U1 pad 17: unconnected-(U1-PH5-Pad17) -> /PH5
- U1 pad 18: unconnected-(U1-PH6-Pad18) -> /PH6
- U1 pad 19: unconnected-(U1-PB0-Pad19) -> /PB0
- U1 pad 2: unconnected-(U1-PE0-Pad2) -> /PE0
- U1 pad 20: unconnected-(U1-PB1-Pad20) -> /PB1
- U1 pad 21: unconnected-(U1-PB2-Pad21) -> /PB2
- U1 pad 22: unconnected-(U1-PB3-Pad22) -> /PB3
- U1 pad 23: unconnected-(U1-PB4-Pad23) -> /PB4
- U1 pad 24: unconnected-(U1-PB5-Pad24) -> /PB5
- U1 pad 25: unconnected-(U1-PB6-Pad25) -> /PB6
- U1 pad 26: unconnected-(U1-PB7-Pad26) -> /PB7
- U1 pad 3: unconnected-(U1-PE1-Pad3) -> /PE1
- U1 pad 35: unconnected-(U1-PL0-Pad35) -> /PL0
- U1 pad 36: unconnected-(U1-PL1-Pad36) -> /PL1
- U1 pad 37: unconnected-(U1-PL2-Pad37) -> /PL2
- U1 pad 38: unconnected-(U1-PL3-Pad38) -> /PL3
- U1 pad 39: unconnected-(U1-PL4-Pad39) -> /PL4
- U1 pad 40: unconnected-(U1-PL5-Pad40) -> /PL5
- U1 pad 41: unconnected-(U1-PL6-Pad41) -> /PL6
- U1 pad 42: unconnected-(U1-PL7-Pad42) -> /PL7
- U1 pad 43: unconnected-(U1-PD0-Pad43) -> /SDA
- U1 pad 44: unconnected-(U1-PD1-Pad44) -> /SCL
- U1 pad 45: unconnected-(U1-PD2-Pad45) -> /RXD1
- U1 pad 5: unconnected-(U1-PE3-Pad5) -> /PE3
- U1 pad 50: unconnected-(U1-PD7-Pad50) -> /PD7
- U1 pad 51: unconnected-(U1-PG0-Pad51) -> /PG0
- U1 pad 52: unconnected-(U1-PG1-Pad52) -> /PG1
- U1 pad 53: unconnected-(U1-PC0-Pad53) -> /PC0
- U1 pad 54: unconnected-(U1-PC1-Pad54) -> /PC1
- U1 pad 55: unconnected-(U1-PC2-Pad55) -> /PC2
- U1 pad 56: unconnected-(U1-PC3-Pad56) -> /PC3
- U1 pad 57: unconnected-(U1-PC4-Pad57) -> /PC4
- U1 pad 58: unconnected-(U1-PC5-Pad58) -> /PC5
- U1 pad 59: unconnected-(U1-PC6-Pad59) -> /PC6
- U1 pad 6: unconnected-(U1-PE4-Pad6) -> /PE4
- U1 pad 60: unconnected-(U1-PC7-Pad60) -> /PC7
- U1 pad 63: unconnected-(U1-PJ0-Pad63) -> /RXD3
- U1 pad 64: unconnected-(U1-PJ1-Pad64) -> /TXD3
- U1 pad 7: unconnected-(U1-PE5-Pad7) -> /PE5
- U1 pad 70: unconnected-(U1-PG2-Pad70) -> /PG2
- U1 pad 71: unconnected-(U1-PA7-Pad71) -> /PA7
- U1 pad 72: unconnected-(U1-PA6-Pad72) -> /PA6
- U1 pad 73: unconnected-(U1-PA5-Pad73) -> /PA5
- U1 pad 74: unconnected-(U1-PA4-Pad74) -> /PA4
- U1 pad 75: unconnected-(U1-PA3-Pad75) -> /PA3
- U1 pad 76: unconnected-(U1-PA2-Pad76) -> /PA2
- U1 pad 77: unconnected-(U1-PA1-Pad77) -> /PA1
- U1 pad 78: unconnected-(U1-PA0-Pad78) -> /PA0
- U1 pad 82: unconnected-(U1-PK7-Pad82) -> /ADC8
- U1 pad 83: unconnected-(U1-PK6-Pad83) -> /ADC9
- U1 pad 84: unconnected-(U1-PK5-Pad84) -> /ADC10
- U1 pad 85: unconnected-(U1-PK4-Pad85) -> /ADC11
- U1 pad 86: unconnected-(U1-PK3-Pad86) -> /ADC12
- U1 pad 87: unconnected-(U1-PK2-Pad87) -> /ADC13
- U1 pad 88: unconnected-(U1-PK1-Pad88) -> /ADC14
- U1 pad 89: unconnected-(U1-PK0-Pad89) -> /ADC15
- U1 pad 90: unconnected-(U1-PF7-Pad90) -> /ADC0
- U1 pad 91: unconnected-(U1-PF6-Pad91) -> /ADC1
- U1 pad 92: unconnected-(U1-PF5-Pad92) -> /ADC2
- U1 pad 93: unconnected-(U1-PF4-Pad93) -> /ADC3
- U1 pad 94: unconnected-(U1-PF3-Pad94) -> /ADC4
- U1 pad 95: unconnected-(U1-PF2-Pad95) -> Net-(J4-Pin_3)
- U1 pad 96: unconnected-(U1-PF1-Pad96) -> Net-(J4-Pin_2)
- U1 pad 97: unconnected-(U1-PF0-Pad97) -> Net-(J4-Pin_1)
Routing:
- net GND: track 0.00 -> 15.5 mm
- net Net-(U5-PC0/XTAL2): track 0.00 -> 6.08 mm
- net Net-(U5-XTAL1): track 0.00 -> 3.84 mm
- net /USB/VUCAP: track 0.00 -> 3.78 mm
- net /USB/UGND: track 0.00 -> 3.78 mm
- net +5V: track 0.00 -> 3.19 mm
