File: New_Atmega 2560/New_Atmega 2560.kicad_sch (KiCad schematic)
At the start: 19 parts, among them IC1 1870_LD11117S50CTR, IC2 MC33269D-5.0, J1 Barrel_Jack_Switch, U1 ATmega2560-16A, Y1 Crystal, Y2 16Hz

Commit message: Add files via upload
Parts:
- added RN1A1, RN1D1: 10k, symbol Device:R
- added RN2B1, RN2C1: 22R, symbol Device:R
- added RN3C1: 1k, symbol Device:R
- added XIO: Conn_02x18_Counter_Clockwise, Connector_PinHeader_2.54mm:PinHeader_2x18_P2.54mm_Vertical, symbol Connector_Generic:Conn_02x18_Counter_Clockwise
- renumbered C3 to C1, C2 to C16, C5 to C2, C4 to C7
Connections:
- net +5V: now also XIO.1 (Pin_1), XIO.2 (Pin_2)
- net GND: now also C16.2, C4.2, C5.2, C6.2, U1.11 (GND), U1.32 (GND), U1.62 (GND), U1.81 (GND), U1.99 (GND)
- net VCC: now reaches U1.10 (VCC), U1.31 (VCC), U1.61 (VCC), U1.80 (VCC)
- net RESET: now reaches U1.30 (~{RESET})
- new net PA1: XIO.4 (Pin_4)
Other:
- moved on the sheet: C16, C4, C5, C6, L1, U1

Commit message: Add files via upload
Parts:
- added ADCH: ADCH, symbol Connector_Generic:Conn_01x08
- added C8, C9: 100n, symbol Device:C
- added J2: Conn_01x08, symbol Connector_Generic:Conn_01x08
- added RN5C, RN5D: 10k, symbol Device:R
- added SW1: SW_Push, symbol Switch:SW_Push
- added U2: LMV358, symbol Amplifier_Operational:LMV358
- added U3: LP2985-3.3, Package_TO_SOT_SMD:SOT-23-5, symbol Regulator_Linear:LP2985-3.3
Connections:
- net +5V: now also C8.1, J2.2 (Pin_2), J2.5 (Pin_5)
- net GND: now also J1.2, XIO.35 (Pin_35), XIO.36 (Pin_36), C8.2, C9.2, J2.6 (Pin_6), J2.7 (Pin_7), RN5D.2, SW1.1
- net RESET: now also J2.3 (Pin_3), SW1.2
- net VIN: now also J2.8 (Pin_8), RN5C.1
- net RXD2: now reaches U1.12 (PH0)
- net TXD2: now reaches U1.13 (PH1)
- net RXD3: now reaches U1.63 (PJ0)
- net TXD3: now reaches U1.64 (PJ1)
- net at U1.82 (PK7): now also ADCH.1 (Pin_1)
- net at U1.83 (PK6): now also ADCH.2 (Pin_2)
- net at U1.84 (PK5): now also ADCH.3 (Pin_3)
- net at U1.85 (PK4): now also ADCH.4 (Pin_4)
- net at U1.86 (PK3): now also ADCH.5 (Pin_5)
- net at U1.87 (PK2): now also ADCH.6 (Pin_6)
- net at U1.88 (PK1): now also ADCH.7 (Pin_7)
- net at U1.89 (PK0): now also ADCH.8 (Pin_8)
- net PA7: now reaches XIO.10 (Pin_10)
- net PC7: now reaches XIO.11 (Pin_11)
- net PC6: now reaches XIO.12 (Pin_12)
- net PC5: now reaches XIO.13 (Pin_13)
- net PC4: now reaches XIO.14 (Pin_14)
- net PC3: now reaches XIO.15 (Pin_15)
- net PC2: now reaches XIO.16 (Pin_16)
- net PC1: now reaches XIO.17 (Pin_17)
- net PC0: now reaches XIO.18 (Pin_18)
- net PD7: now reaches XIO.19 (Pin_19)
- net PG2: now reaches XIO.20 (Pin_20)
- net PG1: now reaches XIO.21 (Pin_21)
- net PG0: now reaches XIO.22 (Pin_22)
- net PL7: now reaches XIO.23 (Pin_23)
- net PL6: now reaches XIO.24 (Pin_24)
- net PL5: now reaches XIO.25 (Pin_25)
- net PL4: now reaches XIO.26 (Pin_26)
- net PL3: now reaches XIO.27 (Pin_27)
- net PL2: now reaches XIO.28 (Pin_28)
- net PL1: now reaches XIO.29 (Pin_29)
- net PL1: now also XIO.33 (Pin_33)
- net PA0: now reaches XIO.3 (Pin_3)
- net PL0: now reaches XIO.30 (Pin_30)
- net PB3: now reaches XIO.31 (Pin_31)
- net PB2: now reaches XIO.32 (Pin_32)
- net PB0: now reaches XIO.34 (Pin_34)
- net PA2: now reaches XIO.5 (Pin_5)
- net PA3: now reaches XIO.6 (Pin_6)
- net PA4: now reaches XIO.7 (Pin_7)
- net PA5: now reaches XIO.8 (Pin_8)
- net PA6: now reaches XIO.9 (Pin_9)
- new net: RN5C.2, RN5D.1
- new net +3V3: J2.4 (Pin_4)
- new net 3V3: U2.2 (-)
- new net CMP: C9.1, U2.3 (+)
Other:
- moved on the sheet: C1, C16, C2, C3, C4, C5, C6, C7, CPC1, D1, IC1, IC2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

Commit message: New Verstion
I add some material
Parts:
- removed Y1: Crystal, symbol Device:Crystal
- added C10: 1u, symbol Device:C
- added C11: C, symbol Device:C
- added D3: CD1206-S01575, symbol Device:D
- added GREEN: ON, symbol Device:LED
- added J3, J4, J5: Conn_01x08, symbol Connector_Generic:Conn_01x08
- added J6: Conn_01x10, symbol Connector_Generic:Conn_01x10
- added J7: Conn_01x06, symbol Connector_Generic:Conn_01x06
- added RN1B, RN1C, RN5A: 10K, symbol Device:R
- added RN3A, RN3B: 1K, symbol Device:R
- added U4: LMV358IDGKR, symbol Amplifier_Operational:LMV358
- added YELLOW: L, symbol Device:LED
- C1, C7: value ~ -> (none)
- U2: value LMV358 -> LMV358IDGKR
- U3: value LP2985-3.3 -> LP2985-33DBVR
- XIO: value Conn_02x18_Counter_Clockwise -> 18x2F-H8.5
- renumbered Y2 to Y1
Connections:
- net +5V: now also U3.1 (VIN), U3.3 (ON/~{OFF}), D3.1 (K), J7.2 (Pin_2), RN1B.1, RN1C.1, RN3A.1, RN5A.1
- net AREF: now also J6.3 (Pin_3)
- net GND: now also U3.2 (GND), C10.2, C11.2, GREEN.1 (K), J6.4 (Pin_4), J7.6 (Pin_6), YELLOW.1 (K)
- net PA0: now also U1.78 (PA0)
- net PA1: now also U1.77 (PA1)
- net PA2: now also U1.76 (PA2)
- net PA3: now also U1.75 (PA3)
- net PA4: now also U1.74 (PA4)
- net PA5: now also U1.73 (PA5)
- net PA6: now also U1.72 (PA6)
- net PA7: now also U1.71 (PA7)
- net PB0: now also U1.19 (PB0)
- net PB2: now also U1.21 (PB2), J7.4 (Pin_4)
- net PB3: now also U1.22 (PB3), J7.1 (Pin_1)
- net PC0: now also U1.53 (PC0)
- net PC1: now also U1.54 (PC1)
- net PC2: now also U1.55 (PC2)
- net PC3: now also U1.56 (PC3)
- net PC4: now also U1.57 (PC4)
- net PC5: now also U1.58 (PC5)
- net PC6: now also U1.59 (PC6)
- net PC7: now also U1.60 (PC7)
- net PD7: now also U1.50 (PD7)
- net PG0: now also U1.51 (PG0)
- net PG1: now also U1.52 (PG1)
- net PG2: now also U1.70 (PG2)
- net PL0: now also U1.35 (PL0)
- net PL1: now also U1.36 (PL1)
- net PL2: now also U1.37 (PL2)
- net PL3: now also U1.38 (PL3)
- net PL4: now also U1.39 (PL4)
- net PL5: now also U1.40 (PL5)
- net PL6: now also U1.41 (PL6)
- net PL7: now also U1.42 (PL7)
- net RESET: now also C11.1, D3.2 (A), J7.5 (Pin_5), RN5A.2
- net RXD2: now also J5.5 (Pin_5)
- net RXD3: now also J5.7 (Pin_7)
- net TXD2: now also J5.6 (Pin_6)
- net TXD3: now also J5.8 (Pin_8)
- net +3v3: now reaches U3.5 (VOUT)
- net +3v3: now also C10.1
- net PG5: now reaches U1.1 (PG5)
- net PG5: now also J3.5 (Pin_5)
- net PH3: now reaches U1.15 (PH3)
- net PH3: now also J3.7 (Pin_7)
- net PH4: now reaches U1.16 (PH4)
- net PH4: now also J3.8 (Pin_8)
- net PH5: now reaches U1.17 (PH5)
- net PH5: now also J6.10 (Pin_10)
- net PH6: now reaches U1.18 (PH6)
- net PH6: now also J6.9 (Pin_9)
- net PE0: now reaches U1.2 (PE0)
- net PE0: now also J3.1 (Pin_1)
- net PB1: now reaches U1.20 (PB1)
- net PB1: now also J7.3 (Pin_3)
- net PB4: now reaches U1.23 (PB4)
- net PB4: now also J6.8 (Pin_8)
- net PB5: now reaches U1.24 (PB5)
- net PB5: now also J6.7 (Pin_7)
- net PB6: now reaches U1.25 (PB6)
- net PB6: now also J6.6 (Pin_6)
- net PB7: now reaches U1.26 (PB7)
- net PB7: now also J6.5 (Pin_5), U4.3 (+)
- net PE1: now reaches U1.3 (PE1)
- net PE1: now also J3.2 (Pin_2)
- net SDA: now reaches U1.43 (PD0)
- net SDA: now also J5.1 (Pin_1), J6.2 (Pin_2), RN1C.2
- net SCL: now reaches U1.44 (PD1)
- net SCL: now also J5.2 (Pin_2), J6.1 (Pin_1), RN1B.2
- net RXD1: now reaches U1.45 (PD2)
- net RXD1: now also J5.3 (Pin_3)
- net PE3: now reaches U1.5 (PE3)
- net PE3: now also J3.6 (Pin_6)
- net PE4: now reaches U1.6 (PE4)
- net PE4: now also J3.3 (Pin_3)
- net PE5: now reaches U1.7 (PE5)
- net PE5: now also J3.4 (Pin_4)
- net ADC8: now reaches ADCH.1 (Pin_1), U1.82 (PK7)
- net ADC9: now reaches ADCH.2 (Pin_2), U1.83 (PK6)
- net ADC10: now reaches ADCH.3 (Pin_3), U1.84 (PK5)
- net ADC11: now reaches ADCH.4 (Pin_4), U1.85 (PK4)
- net ADC12: now reaches ADCH.5 (Pin_5), U1.86 (PK3)
- net ADC13: now reaches ADCH.6 (Pin_6), U1.87 (PK2)
- net ADC14: now reaches ADCH.7 (Pin_7), U1.88 (PK1)
- net ADC15: now reaches ADCH.8 (Pin_8), U1.89 (PK0)
- net ADC0: now reaches U1.90 (PF7)
- net ADC0: now also J4.8 (Pin_8)
- net ADC1: now reaches U1.91 (PF6)
- net ADC1: now also J4.7 (Pin_7)
- net ADC2: now reaches U1.92 (PF5)
- net ADC2: now also J4.6 (Pin_6)
- net ADC3: now reaches U1.93 (PF4)
- net ADC3: now also J4.5 (Pin_5)
- net ADC4: now reaches U1.94 (PF3)
- net ADC4: now also J4.4 (Pin_4)
- net ADC5: now reaches U1.95 (PF2)
- net ADC5: now also J4.3 (Pin_3)
- net ADC6: now reaches U1.96 (PF1)
- net ADC6: now also J4.2 (Pin_2)
- net ADC7: now reaches U1.97 (PF0)
- net ADC7: now also J4.1 (Pin_1)
- new net: RN3B.2, YELLOW.2 (A)
- new net: GREEN.2 (A), RN3A.2
- new net L13: RN3B.1, U4.1, U4.2 (-)
- new net TXD1: J5.4 (Pin_4)
Other:
- added sheet USB (usb.kicad_sch)
- moved on the sheet: C16, C4, C5, C6, L1, U3

Commit message: Update
update the material
Parts:
- C10, C11, C8, C9: footprint (none) -> Capacitor_SMD:C_0603_1608Metric
- GREEN1: renamed from GREEN; footprint (none) -> LED_SMD:LED_PLCC_2835
- IC2: footprint (none) -> Library:TO229P990X238-4N
- R1: footprint (none) -> Resistor_SMD:R_0603_1608Metric
- YELLOW1: renamed from YELLOW; footprint (none) -> LED_SMD:LED_PLCC_2835
- renumbered ADCH to ADCH1, RN1B to RN1B1, RN1C to RN1C1, RN3A to RN3A1, RN3B to RN3B1, RN5A to RN5A1, RN5C to RN5C1, RN5D to RN5D1, XIO to XIO1
Changed lines of the file:
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@@
 			)
 		)
-		(property "Footprint" ""
+		(property "Footprint" "Capacitor_SMD:C_0603_1608Metric"
 			(at 117.8052 186.69 0)
 			(hide yes)
@@
 			)
 		)
-		(property "Footprint" ""
+		(property "Footprint" "Capacitor_SMD:C_0603_1608Metric"
 			(at 234.6452 36.83 0)
 			(hide yes)
@@
 		(in_pos_files yes)
 		(dnp no)
-		(property "Reference" "RN1B"
+		(property "Reference" "RN1B1"
 			(at 269.748 28.956 90)
 			(show_name no)
@@
 			(project "New_Atmega 2560"
 				(path "/f123d371-868a-48f0-9f6c-663b3f4e9af5"
-					(reference "RN1B")
+					(reference "RN1B1")
 					(unit 1)
 				)
@@
 		(in_pos_files yes)
 		(dnp no)
-		(property "Reference" "RN5A"
+		(property "Reference" "RN5A1"
 			(at 243.586 25.146 90)
 			(show_name no)
@@
 			(project "New_Atmega 2560"
 				(path "/f123d371-868a-48f0-9f6c-663b3f4e9af5"
-					(reference "RN5A")
+					(reference "RN5A1")
 					(unit 1)
 				)
@@
 			)
 		)
-		(property "Footprint" ""
+		(property "Footprint" "Library:TO229P990X238-4N"
 			(at 76.2 36.83 0)
 			(hide yes)
@@
 			)
 		)
-		(property "Footprint" ""
+		(property "Footprint" "Capacitor_SMD:C_0603_1608Metric"
 			(at 22.5552 181.61 0)
 			(hide yes)
@@
 		(in_pos_files yes)
 		(dnp no)
-		(property "Reference" "RN1C"
+		(property "Reference" "RN1C1"
 			(at 276.352 28.956 90)
 			(show_name no)
@@
 			(project "New_Atmega 2560"
 				(path "/f123d371-868a-48f0-9f6c-663b3f4e9af5"
-					(reference "RN1C")
+					(reference "RN1C1")
 					(unit 1)
 				)
@@
 		(in_pos_files yes)
 		(dnp no)
-		(property "Reference" "YELLOW"
+		(property "Reference" "YELLOW1"
 			(at 208.28 21.59 0)
 			(show_name no)
@@
 			)
 		)
-		(property "Footprint" ""
+		(property "Footprint" "LED_SMD:LED_PLCC_2835"
 			(at 209.55 24.13 0)
 			(hide yes)
@@
 			(project "New_Atmega 2560"
 				(path "/f123d371-868a-48f0-9f6c-663b3f4e9af5"
-					(reference "YELLOW")
+					(reference "YELLOW1")
 					(unit 1)
 				)
@@
 		(in_pos_files yes)
 		(dnp no)
-		(property "Reference" "RN3A"
+		(property "Reference" "RN3A1"
 			(at 200.406 16.256 90)
 			(show_name no)
@@
 			(project "New_Atmega 2560"
 				(path "/f123d371-868a-48f0-9f6c-663b3f4e9af5"
-					(reference "RN3A")
+					(reference "RN3A1")
 					(unit 1)
 				)
@@
 		(in_pos_files yes)
 		(dnp no)
-		(property "Reference" "GREEN"
+		(property "Reference" "GREEN1"
 			(at 208.534 16.51 0)
 			(show_name no)
@@
 			)
 		)
-		(property "Footprint" ""
+		(property "Footprint" "LED_SMD:LED_PLCC_2835"
 			(at 209.55 19.05 0)
 			(hide yes)
@@
 			(project "New_Atmega 2560"
 				(path "/f123d371-868a-48f0-9f6c-663b3f4e9af5"
-					(reference "GREEN")
+					(reference "GREEN1")
 					(unit 1)
 				)
@@
 		(in_pos_files yes)
 		(dnp no)
-		(property "Reference" "RN5C"
+		(property "Reference" "RN5C1"
 			(at 53.34 149.352 90)
 			(show_name no)
@@
 			(project "New_Atmega 2560"
 				(path "/f123d371-868a-48f0-9f6c-663b3f4e9af5"
-					(reference "RN5C")
+					(reference "RN5C1")
 					(unit 1)
 				)
@@
 			)
 		)
-		(property "Footprint" ""
+		(property "Footprint" "Resistor_SMD:R_0603_1608Metric"
 			(at 54.102 72.39 90)
 			(hide yes)
@@
 		(in_pos_files yes)
 		(dnp no)
-		(property "Reference" "ADCH"
+		(property "Reference" "ADCH1"
 			(at 99.568 95.504 0)
 			(show_name no)
@@
 			(project "New_Atmega 2560"
 				(path "/f123d371-868a-48f0-9f6c-663b3f4e9af5"
-					(reference "ADCH")
+					(reference "ADCH1")
 					(unit 1)
 				)
@@
 		(in_pos_files yes)
 		(dnp no)
-		(property "Reference" "RN3B"
+		(property "Reference" "RN3B1"
 			(at 200.406 21.844 90)
 			(show_name no)
@@
 			(project "New_Atmega 2560"
 				(path "/f123d371-868a-48f0-9f6c-663b3f4e9af5"
-					(reference "RN3B")
+					(reference "RN3B1")
 					(unit 1)
 				)
@@
 		(in_pos_files yes)
 		(dnp no)
-		(property "Reference" "XIO"
+		(property "Reference" "XIO1"
 			(at 27.432 120.65 0)
 			(show_name no)
@@
 			(project "New_Atmega 2560"
 				(path "/f123d371-868a-48f0-9f6c-663b3f4e9af5"
-					(reference "XIO")
+					(reference "XIO1")
 					(unit 1)
 				)
@@
 		(in_pos_files yes)
 		(dnp no)
-		(property "Reference" "RN5D"
+		(property "Reference" "RN5D1"
 			(at 53.34 159.258 90)
 			(show_name no)
@@
 			(project "New_Atmega 2560"
 				(path "/f123d371-868a-48f0-9f6c-663b3f4e9af5"
-					(reference "RN5D")
+					(reference "RN5D1")
 					(unit 1)
 				)
@@
 			)
 		)
-		(property "Footprint" ""
+		(property "Footprint" "Capacitor_SMD:C_0603_1608Metric"
 			(at 69.5452 158.75 0)
 			(hide yes)

Commit message: New V
Parts:
- D3: footprint (none) -> Diode_SMD:D_MiniMELF
- IC1: footprint (none) -> Package_TO_SOT_SMD:SOT-223-3_TabPin2
- J2, J3, J4, J5, J6, J7: footprint (none) -> Connector_PinHeader_2.54mm:PinHeader_2x02_P2.54mm_Vertical
- RN1A1, RN1B1, RN1C1, RN1D1, RN2B1, RN2C1, RN3A1, RN3B1, RN3C1, RN5A1, RN5C1, RN5D1: footprint (none) -> Resistor_THT:R_Array_SIP8
Changed lines of the file:
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@@
 			)
 		)
-		(property "Footprint" ""
+		(property "Footprint" "Connector_PinHeader_2.54mm:PinHeader_2x02_P2.54mm_Vertical"
 			(at 179.07 116.84 0)
 			(hide yes)
@@
 			)
 		)
-		(property "Footprint" ""
+		(property "Footprint" "Package_TO_SOT_SMD:SOT-223-3_TabPin2"
 			(at 73.66 17.78 0)
 			(hide yes)
@@
 			)
 		)
-		(property "Footprint" ""
+		(property "Footprint" "Diode_SMD:D_MiniMELF"
 			(at 248.92 21.59 0)
 			(hide yes)
@@
 			)
 		)
-		(property "Footprint" ""
+		(property "Footprint" "Connector_PinHeader_2.54mm:PinHeader_2x02_P2.54mm_Vertical"
 			(at 184.15 68.58 0)
 			(hide yes)
@@
 			)
 		)
-		(property "Footprint" ""
+		(property "Footprint" "Connector_PinHeader_2.54mm:PinHeader_2x02_P2.54mm_Vertical"
 			(at 179.07 139.7 0)
 			(hide yes)
@@
 			)
 		)
-		(property "Footprint" ""
+		(property "Footprint" "Connector_PinHeader_2.54mm:PinHeader_2x02_P2.54mm_Vertical"
 			(at 49.53 184.15 0)
 			(hide yes)
@@
 			)
 		)
-		(property "Footprint" ""
+		(property "Footprint" "Connector_PinHeader_2.54mm:PinHeader_2x02_P2.54mm_Vertical"
 			(at 179.07 162.56 0)
 			(hide yes)
@@
 			)
 		)
-		(property "Footprint" ""
+		(property "Footprint" "Resistor_THT:R_Array_SIP8"
 			(at 264.922 25.4 90)
 			(hide yes)
@@
 			)
 		)
-		(property "Footprint" ""
+		(property "Footprint" "Resistor_THT:R_Array_SIP8"
 			(at 239.522 21.59 90)
 			(hide yes)
@@
 			)
 		)
-		(property "Footprint" ""
+		(property "Footprint" "Resistor_THT:R_Array_SIP8"
 			(at 111.76 36.068 90)
 			(hide yes)
@@
 			)
 		)
-		(property "Footprint" ""
+		(property "Footprint" "Connector_PinHeader_2.54mm:PinHeader_2x02_P2.54mm_Vertical"
 			(at 228.6 54.61 0)
 			(hide yes)
@@
 			)
 		)
-		(property "Footprint" ""
+		(property "Footprint" "Resistor_THT:R_Array_SIP8"
 			(at 111.76 30.988 90)
 			(hide yes)
@@
 			)
 		)
-		(property "Footprint" ""
+		(property "Footprint" "Resistor_THT:R_Array_SIP8"
 			(at 271.272 25.4 90)
 			(hide yes)
@@
 			)
 		)
-		(property "Footprint" ""
+		(property "Footprint" "Resistor_THT:R_Array_SIP8"
 			(at 111.76 15.748 90)
 			(hide yes)
@@
 			)
 		)
-		(property "Footprint" ""
+		(property "Footprint" "Resistor_THT:R_Array_SIP8"
 			(at 198.12 20.828 90)
 			(hide yes)
@@
 			)
 		)
-		(property "Footprint" ""
+		(property "Footprint" "Resistor_THT:R_Array_SIP8"
 			(at 49.022 144.78 90)
 			(hide yes)
@@
 			)
 		)
-		(property "Footprint" ""
+		(property "Footprint" "Resistor_THT:R_Array_SIP8"
 			(at 111.76 20.828 90)
 			(hide yes)
@@
 			)
 		)
-		(property "Footprint" ""
+		(property "Footprint" "Resistor_THT:R_Array_SIP8"
 			(at 198.12 25.908 90)
 			(hide yes)
@@
 			)
 		)
-		(property "Footprint" ""
+		(property "Footprint" "Resistor_THT:R_Array_SIP8"
 			(at 49.022 156.21 90)
 			(hide yes)
@@
 			)
 		)
-		(property "Footprint" ""
+		(property "Footprint" "Resistor_THT:R_Array_SIP8"
 			(at 111.76 25.908 90)
 			(hide yes)

Commit message: Arduino Mega 2560 upload
Parts:
- ADCH1: footprint (none) -> Connector_PinHeader_2.54mm:PinHeader_1x08_P2.54mm_Vertical
- SW1: footprint (none) -> Button_Switch_SMD:SW_SPST_Omron_B3FS-1xxx
- U2, U4: footprint (none) -> Package_SO:MSOP-8_3x3mm_P0.65mm
- Y1: footprint (none) -> Crystal:Crystal_SMD_HC49-SD
- YELLOW1: footprint LED_SMD:LED_PLCC_2835 -> LED_SMD:LED_0805_2012Metric
Changed lines of the file:
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@@
 			)
 		)
-		(property "Footprint" ""
+		(property "Footprint" "Package_SO:MSOP-8_3x3mm_P0.65mm"
 			(at 86.36 146.05 0)
 			(hide yes)
@@
 			)
 		)
-		(property "Footprint" ""
+		(property "Footprint" "Crystal:Crystal_SMD_HC49-SD"
 			(at 80.01 71.12 0)
 			(hide yes)
@@
 			)
 		)
-		(property "Footprint" "LED_SMD:LED_PLCC_2835"
+		(property "Footprint" "LED_SMD:LED_0805_2012Metric"
 			(at 209.55 24.13 0)
 			(hide yes)
@@
 			)
 		)
-		(property "Footprint" ""
+		(property "Footprint" "Connector_PinHeader_2.54mm:PinHeader_1x08_P2.54mm_Vertical"
 			(at 104.14 96.52 0)
 			(hide yes)
@@
 			)
 		)
-		(property "Footprint" ""
+		(property "Footprint" "Package_SO:MSOP-8_3x3mm_P0.65mm"
 			(at 181.61 24.13 0)
 			(hide yes)
@@
 			)
 		)
-		(property "Footprint" ""
+		(property "Footprint" "Button_Switch_SMD:SW_SPST_Omron_B3FS-1xxx"
 			(at 25.4 186.69 0)
 			(hide yes)
