File: New_Atmega 2560/New_Atmega 2560.kicad_sch (KiCad schematic)
At the start: 49 parts, among them IC1 1870_LD11117S50CTR, IC2 MC33269D-5.0, J1 Barrel_Jack_Switch, J2 Conn_01x08, J3 Conn_01x08, J4 Conn_01x08, J5 Conn_01x08, J6 Conn_01x10, J7 Conn_01x06, SW1 SW_Push, U1 ATmega2560-16A, U2 LMV358IDGKR, U3 LP2985-33DBVR, U4 LMV358IDGKR, Y1 16Hz

Commit message: PCB電路圖設計
Connections:
- net +3v3 is gone; now on net +3V3: C10.1, U3.5 (VOUT)
- net AVCC is gone; now on net +5V: U1.100 (AVCC)
- net VCC is gone; now on net +5V: U1.10 (VCC), U1.31 (VCC), U1.61 (VCC), U1.80 (VCC)
- net XTL1 is gone; now on net XTAL1: U1.34 (XTAL1)
- net XTL2 is gone; now on net XTAL2: U1.33 (XTAL2)
