File: New_Atmega 2560/usb.kicad_sch (KiCad schematic)
At the start: 27 parts, among them J8 Conn_PIC_ICSP_ICD, J9 Conn_02x02_Counter_Clockwise, P1 USB_C_Plug_USB2.0, U5 ATmega16U2-M, Y2 Crystal

Commit message: Update
update the material
Parts:
- C12, C13, C14, C15, C17: footprint (none) -> Capacitor_SMD:C_0603_1608Metric
- C18: footprint (none) -> Capacitor_SMD:C_0603_1608Metric_Pad1.08x0.95mm_HandSolder
- F1: footprint FUSER_MF-MSMF050 -> MF-MSMF050:FUSER_MF-MSMF050
- FB1: footprint L0805 -> mh2029-300y:L0805
- P1: footprint (none) -> Connector_USB:USB_C_Plug_Molex_105444
- R2, R3, R4, R5: footprint (none) -> Resistor_SMD:R_0603_1608Metric
- RX1: renamed from RX; footprint (none) -> LED_SMD:LED_PLCC_2835
- TX1: renamed from TX; footprint (none) -> LED_SMD:LED_PLCC_2835
- renumbered RN3D to RN3D1, RN4A to RN4A1, RN4B to RN4B1, RN4C to RN4C2
Connections:
- net GND: now also C18.1
Changed lines of the file:
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@@
 	(wire
 		(pts
+			(xy 74.93 54.61) (xy 74.93 55.88)
+		)
+		(stroke
+			(width 0)
+			(type default)
+		)
+	)
+	(wire
+		(pts
 			(xy 97.79 142.24) (xy 57.15 142.24)
 		)
@@
 		(dnp no)
 		(fields_autoplaced yes)
-		(property "Reference" "RX"
+		(property "Reference" "RX1"
 			(at 186.3725 113.03 0)
 			(show_name no)
@@
 			)
 		)
-		(property "Footprint" ""
+		(property "Footprint" "LED_SMD:LED_PLCC_2835"
 			(at 187.96 119.38 0)
 			(hide yes)
@@
 			(project "New_Atmega 2560"
 				(path "/f123d371-868a-48f0-9f6c-663b3f4e9af5/afb03c50-fd2e-450d-8b7a-da4257288ef8"
-					(reference "RX")
+					(reference "RX1")
 					(unit 1)
 				)
@@
 			)
 		)
-		(property "Footprint" ""
+		(property "Footprint" "Resistor_SMD:R_0603_1608Metric"
 			(at 97.79 100.838 90)
 			(hide yes)
@@
 			)
 		)
-		(property "Footprint" ""
+		(property "Footprint" "Capacitor_SMD:C_0603_1608Metric"
 			(at 184.15 74.93 0)
 			(hide yes)
@@
 			)
 		)
-		(property "Footprint" ""
+		(property "Footprint" "Capacitor_SMD:C_0603_1608Metric"
 			(at 97.79 119.38 0)
 			(hide yes)
@@
 			)
 		)
-		(property "Footprint" ""
+		(property "Footprint" "Resistor_SMD:R_0603_1608Metric"
 			(at 104.902 86.36 90)
 			(hide yes)
@@
 			)
 		)
-		(property "Footprint" ""
+		(property "Footprint" "Resistor_SMD:R_0603_1608Metric"
 			(at 118.872 64.77 90)
 			(hide yes)
@@
 			)
 		)
-		(property "Footprint" ""
+		(property "Footprint" "Resistor_SMD:R_0603_1608Metric"
 			(at 97.79 105.918 90)
 			(hide yes)
@@
 		(in_pos_files yes)
 		(dnp no)
-		(property "Reference" "RN4C"
+		(property "Reference" "RN4C2"
 			(at 198.12 117.094 90)
 			(show_name no)
@@
 			(project "New_Atmega 2560"
 				(path "/f123d371-868a-48f0-9f6c-663b3f4e9af5/afb03c50-fd2e-450d-8b7a-da4257288ef8"
-					(reference "RN4C")
+					(reference "RN4C2")
 					(unit 1)
 				)
@@
 			)
 		)
-		(property "Footprint" "L0805"
+		(property "Footprint" "mh2029-300y:L0805"
 			(at 48.26 99.06 0)
 			(hide yes)
@@
 			)
 		)
-		(property "Footprint" "FUSER_MF-MSMF050"
+		(property "Footprint" "MF-MSMF050:FUSER_MF-MSMF050"
 			(at 64.77 64.77 0)
 			(hide yes)
@@
 			)
 		)
-		(property "Footprint" ""
+		(property "Footprint" "Connector_USB:USB_C_Plug_Molex_105444"
 			(at 27.94 68.58 0)
 			(hide yes)
@@
 		(dnp no)
 		(fields_autoplaced yes)
-		(property "Reference" "TX"
+		(property "Reference" "TX1"
 			(at 186.3725 123.19 0)
 			(show_name no)
@@
 			)
 		)
-		(property "Footprint" ""
+		(property "Footprint" "LED_SMD:LED_PLCC_2835"
 			(at 187.96 129.54 0)
 			(hide yes)
@@
 			(project "New_Atmega 2560"
 				(path "/f123d371-868a-48f0-9f6c-663b3f4e9af5/afb03c50-fd2e-450d-8b7a-da4257288ef8"
-					(reference "TX")
+					(reference "TX1")
 					(unit 1)
 				)
@@
 		(dnp no)
 		(fields_autoplaced yes)
-		(property "Reference" "RN3D"
+		(property "Reference" "RN3D1"
 			(at 186.69 140.9699 0)
 			(show_name no)
@@
 			(project "New_Atmega 2560"
 				(path "/f123d371-868a-48f0-9f6c-663b3f4e9af5/afb03c50-fd2e-450d-8b7a-da4257288ef8"
-					(reference "RN3D")
+					(reference "RN3D1")
 					(unit 1)
 				)
@@
 		(in_pos_files yes)
 		(dnp no)
-		(property "Reference" "RN4A"
+		(property "Reference" "RN4A1"
 			(at 180.34 104.394 90)
 			(show_name no)
@@
 			(project "New_Atmega 2560"
 				(path "/f123d371-868a-48f0-9f6c-663b3f4e9af5/afb03c50-fd2e-450d-8b7a-da4257288ef8"
-					(reference "RN4A")
+					(reference "RN4A1")
 					(unit 1)
 				)
@@
 			)
 		)
-		(property "Footprint" ""
+		(property "Footprint" "Capacitor_SMD:C_0603_1608Metric"
 			(at 198.12 134.62 0)
 			(hide yes)
@@
 		(in_pos_files yes)
 		(dnp no)
-		(property "Reference" "RN4B"
+		(property "Reference" "RN4B1"
 			(at 180.34 99.314 90)
 			(show_name no)
@@
 			(project "New_Atmega 2560"
 				(path "/f123d371-868a-48f0-9f6c-663b3f4e9af5/afb03c50-fd2e-450d-8b7a-da4257288ef8"
-					(reference "RN4B")
+					(reference "RN4B1")
 					(unit 1)
 				)
@@
 			)
 		)
-		(property "Footprint" ""
+		(property "Footprint" "Capacitor_SMD:C_0603_1608Metric"
 			(at 87.63 90.17 0)
 			(hide yes)
@@
 			)
 		)
-		(property "Footprint" ""
+		(property "Footprint" "Capacitor_SMD:C_0603_1608Metric"
 			(at 87.63 82.55 0)
 			(hide yes)
@@
 			)
 		)
-		(property "Footprint" ""
+		(property "Footprint" "Capacitor_SMD:C_0603_1608Metric_Pad1.08x0.95mm_HandSolder"
 			(at 74.93 59.69 0)
 			(hide yes)
@@
 					(unit 1)
 				)
+			)
+		)
+	)
+	(symbol
+		(lib_id "power:GND")
+		(at 74.93 54.61 180)
+		(unit 1)
+		(body_style 1)
+		(exclude_from_sim no)
+		(in_bom yes)
+		(on_board yes)
+		(in_pos_files yes)
+		(dnp no)
+		(fields_autoplaced yes)
+		(property "Reference" "#PWR039"
+			(at 74.93 48.26 0)
+			(hide yes)
+			(show_name no)
+			(do_not_autoplace no)
+			(effects
+				(font
+					(size 1.27 1.27)
+				)
+			)
+		)
+		(property "Value" "GND"
+			(at 74.93 49.53 0)
+			(show_name no)
+			(do_not_autoplace no)
+			(effects
+				(font
+					(size 1.27 1.27)
+				)
+			)
+		)
+		(property "Footprint" ""
+			(at 74.93 54.61 0)
+			(hide yes)
+			(show_name no)
+			(do_not_autoplace no)
+			(effects
+				(font
+					(size 1.27 1.27)
+				)
+			)
+		)
+		(property "Datasheet" ""
+			(at 74.93 54.61 0)
+			(hide yes)
+			(show_name no)
+			(do_not_autoplace no)
+			(effects
+				(font
+					(size 1.27 1.27)
+				)
+			)
+		)
+		(property "Description" "Power symbol creates a global label with name \"GND\" , ground"
+			(at 74.93 54.61 0)
+			(hide yes)
+			(show_name no)
+			(do_not_autoplace no)
+			(effects
+				(font
+					(size 1.27 1.27)
+				)
+			)
+		)
+		(pin "1"
+		)
+		(instances
+			(project "New_Atmega 2560"
+				(path "/f123d371-868a-48f0-9f6c-663b3f4e9af5/afb03c50-fd2e-450d-8b7a-da4257288ef8"
+					(reference "#PWR039")
+					(unit 1)
+				)

Commit message: New V
Parts:
- D2: footprint (none) -> Diode_SMD:D_MiniMELF
- J8, J9: footprint (none) -> Connector_PinHeader_2.54mm:PinHeader_2x02_P2.54mm_Vertical
- RN3D1, RN4A1, RN4B1, RN4C1, RN4C2: footprint (none) -> Resistor_THT:R_Array_SIP8
Changed lines of the file:
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@@
 			)
 		)
-		(property "Footprint" ""
+		(property "Footprint" "Connector_PinHeader_2.54mm:PinHeader_2x02_P2.54mm_Vertical"
 			(at 99.06 46.99 0)
 			(hide yes)
@@
 			)
 		)
-		(property "Footprint" ""
+		(property "Footprint" "Resistor_THT:R_Array_SIP8"
 			(at 200.66 121.158 90)
 			(hide yes)
@@
 			)
 		)
-		(property "Footprint" ""
+		(property "Footprint" "Diode_SMD:D_MiniMELF"
 			(at 127 64.77 0)
 			(hide yes)
@@
 			)
 		)
-		(property "Footprint" ""
+		(property "Footprint" "Connector_PinHeader_2.54mm:PinHeader_2x02_P2.54mm_Vertical"
 			(at 205.74 93.98 0)
 			(hide yes)
@@
 			)
 		)
-		(property "Footprint" ""
+		(property "Footprint" "Resistor_THT:R_Array_SIP8"
 			(at 200.66 130.048 90)
 			(hide yes)
@@
 			)
 		)
-		(property "Footprint" ""
+		(property "Footprint" "Resistor_THT:R_Array_SIP8"
 			(at 182.372 142.24 90)
 			(hide yes)
@@
 			)
 		)
-		(property "Footprint" ""
+		(property "Footprint" "Resistor_THT:R_Array_SIP8"
 			(at 182.88 108.458 90)
 			(hide yes)
@@
 			)
 		)
-		(property "Footprint" ""
+		(property "Footprint" "Resistor_THT:R_Array_SIP8"
 			(at 182.88 103.378 90)
 			(hide yes)

Commit message: Arduino Mega 2560 upload
Parts:
- R6, R7: footprint (none) -> Resistor_SMD:R_0603_1608Metric
- Y2: value Crystal -> CSTCE16M0V53-R0; footprint (none) -> Crystal:Crystal_SMD_Murata_CSTxExxV-3Pin_3.2x1.3mm
Changed lines of the file:
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@@
 			)
 		)
-		(property "Footprint" ""
+		(property "Footprint" "Resistor_SMD:R_0603_1608Metric"
 			(at 61.722 102.87 90)
 			(hide yes)
@@
 			)
 		)
-		(property "Footprint" ""
+		(property "Footprint" "Resistor_SMD:R_0603_1608Metric"
 			(at 70.612 102.87 90)
 			(hide yes)
@@
 			)
 		)
-		(property "Value" "Crystal"
+		(property "Value" "CSTCE16M0V53-R0"
 			(at 118.11 87.6299 90)
 			(show_name no)
@@
 			)
 		)
-		(property "Footprint" ""
+		(property "Footprint" "Crystal:Crystal_SMD_Murata_CSTxExxV-3Pin_3.2x1.3mm"
 			(at 114.3 86.36 0)
 			(hide yes)
