File: Atmega 2560/Atmega 2560.kicad_sch (KiCad schematic)
At the start: 20 parts, among them IC1 MC33269ST-5.0T3, IC2 MC33269D-5.0, J1 Conn_02x06_Row_Letter_First, J2 Barrel_Jack_Switch, SW1 SW_Push, U1 ATmega2560-16A, Y1 16Hz, Y2 Crystal

Commit message: Add files via upload
Parts:
- added C10, C11, C12, C13, C14: C, symbol Device:C
- added D2 (x2): LED, symbol Device:LED
- added JP1, JP2: SolderJumper_2_Open, symbol Jumper:SolderJumper_2_Open
- added R3 (x2), R4 (x2), R5, R6: R, symbol Device:R
- added U2: ~, symbol PIN:JP
- added Y3, Y4: Crystal, symbol Device:Crystal
Connections:
- net GND is gone; now on net +5V: C1.2, C2.2, C3.2, C4.2, C5.2, C6.2, IC1.1, IC2.1 (ADJ), SW1.2
- net +5V: now also C11.1, C12.1, C13.2, C14.2, JP2.2 (B), R3.1, R4.2, R5.1, R6.1, U2.1 (JP1), U2.2 (JP2), U2.3 (JP3), U2.4 (JP4)
- new net: C11.2, Y3.2
- new net: C13.1, Y4.2
- new net: C12.2, Y3.1
- new net: C10.1, JP2.1 (A)
- new net: C10.2, JP1.1 (A), JP1.2 (B)
- new net: D2.2 (A), R4.1
- new net: D2.2 (A), R3.2
- new net: C14.1, Y4.1
