File: New_CPLD_Digtal_Clock_type-c_Battery/New_CPLD_Digtal_Clock_type-c_Battery.kicad_pcb (KiCad board)
At the start: 2 copper layers, 0 parts

Commit message: Add files via upload
Parts:
- added C1: 10uF, Capacitor_SMD:C_0201_0603Metric, F.Cu at (58.0, 56.1)
- added C2: 0.1uF, Capacitor_SMD:C_0201_0603Metric, F.Cu at (58.0, 57.9)
- added C3: 0.1uF, Capacitor_SMD:C_0201_0603Metric, F.Cu at (58.0, 59.6)
- added C4: 0.1uF, Capacitor_SMD:C_0201_0603Metric, F.Cu at (58.0, 61.4)
- added C5: 0.1uF, Capacitor_SMD:C_0201_0603Metric, F.Cu at (58.0, 63.1)
- added C6: 0.1uF, Capacitor_SMD:C_0201_0603Metric, F.Cu at (58.0, 64.9)
- added C7: 0.1uF, Capacitor_SMD:C_0201_0603Metric, F.Cu at (58.0, 66.6)
- added C8: 10uF, Capacitor_SMD:C_0201_0603Metric, F.Cu at (60.4, 56.1)
- added C9: 0.1uF, Capacitor_SMD:C_0201_0603Metric, F.Cu at (60.4, 57.9)
- added D1: LED, LED_SMD:LED_PLCC_2835, F.Cu at (73.8, 43.2)
- added D2: LED, LED_SMD:LED_PLCC_2835, F.Cu at (73.8, 47.5)
- added D3: LED, LED_SMD:LED_PLCC_2835, F.Cu at (73.8, 51.9)
- added J1: Conn_02x05_Odd_Even, Connector_IDC:IDC-Header_2x03_P2.54mm_Vertical, F.Cu at (50.0, 47.1)
- added J2: Conn_01x15, Connector_PinHeader_1.00mm:PinHeader_1x15_P1.00mm_Vertical, F.Cu at (46.4, 59.9)
- added J3: Conn_01x15, Connector_PinHeader_1.00mm:PinHeader_1x15_P1.00mm_Vertical, F.Cu at (49.7, 59.9)
- added P1: USB_C_Plug_USB2.0, Connector_USB:USB_C_Receptacle_GCT_USB4125-xx-x-0190_6P_TopMnt_Horizontal, F.Cu at (70.0, 66.6)
- added Q1: CS9013, Package_TO_SOT_THT:TO-92L, F.Cu at (40.2, 44.3)
- added Q2: CS9013, Package_TO_SOT_THT:TO-92L, F.Cu at (40.2, 49.9)
- added Q3: CS9013, Package_TO_SOT_THT:TO-92L, F.Cu at (40.2, 55.6)
- added Q4: CS9013, Package_TO_SOT_THT:TO-92L, F.Cu at (40.2, 61.2)
- added Q5: FS8205A, FS8205A:SOP65P640X120-8N, F.Cu at (49.9, 77.5)
- added R1: 1k, Resistor_SMD:R_0201_0603Metric, F.Cu at (60.4, 59.6)
- added R10: 220, Resistor_THT:R_Axial_DIN0207_L6.3mm_D2.5mm_P10.16mm_Horizontal, F.Cu at (15.9, 38.5)
- added R11: 220, Resistor_THT:R_Axial_DIN0207_L6.3mm_D2.5mm_P10.16mm_Horizontal, F.Cu at (15.9, 42.6)
- added R12: 220, Resistor_THT:R_Axial_DIN0207_L6.3mm_D2.5mm_P10.16mm_Horizontal, F.Cu at (15.9, 46.6)
- added R13: 220, Resistor_THT:R_Axial_DIN0207_L6.3mm_D2.5mm_P10.16mm_Horizontal, F.Cu at (15.9, 50.7)
- added R14: 2.2k, Resistor_THT:R_Axial_DIN0207_L6.3mm_D2.5mm_P10.16mm_Horizontal, F.Cu at (15.9, 54.7)
- added R15: 2.2k, Resistor_THT:R_Axial_DIN0207_L6.3mm_D2.5mm_P10.16mm_Horizontal, F.Cu at (15.9, 58.8)
- added R16: 2.2k, Resistor_THT:R_Axial_DIN0207_L6.3mm_D2.5mm_P10.16mm_Horizontal, F.Cu at (15.9, 62.8)
- added R17: 2.2k, Resistor_THT:R_Axial_DIN0207_L6.3mm_D2.5mm_P10.16mm_Horizontal, F.Cu at (15.9, 66.9)
- added R18: 220, Resistor_THT:R_Axial_DIN0207_L6.3mm_D2.5mm_P10.16mm_Horizontal, F.Cu at (15.9, 70.9)
- added R19: 220, Resistor_THT:R_Axial_DIN0207_L6.3mm_D2.5mm_P10.16mm_Horizontal, F.Cu at (15.9, 75.0)
- added R2: 4.7k, Resistor_SMD:R_0201_0603Metric, F.Cu at (60.4, 61.4)
- added R20: 220, Resistor_THT:R_Axial_DIN0207_L6.3mm_D2.5mm_P10.16mm_Horizontal, F.Cu at (15.9, 79.0)
- added R21: 1k, Resistor_SMD:R_0201_0603Metric, F.Cu at (62.9, 56.1)
- added R22: 1k, Resistor_SMD:R_0201_0603Metric, F.Cu at (62.9, 57.9)
- added R23: 100, Resistor_SMD:R_0201_0603Metric, F.Cu at (62.9, 59.6)
- added R25: 1k, Resistor_SMD:R_0201_0603Metric, F.Cu at (62.9, 61.4)
- added R26: 1.2k, Resistor_SMD:R_0201_0603Metric, F.Cu at (62.9, 63.1)
- added R3: 4.7k, Resistor_SMD:R_0201_0603Metric, F.Cu at (60.4, 63.1)
- added R4: 4.7k, Resistor_SMD:R_0201_0603Metric, F.Cu at (60.4, 64.9)
- added R5: 220, Resistor_SMD:R_0201_0603Metric, F.Cu at (60.4, 66.6)
- added R6: 220, Resistor_THT:R_Axial_DIN0207_L6.3mm_D2.5mm_P10.16mm_Horizontal, F.Cu at (15.9, 22.3)
- added R7: 220, Resistor_THT:R_Axial_DIN0207_L6.3mm_D2.5mm_P10.16mm_Horizontal, F.Cu at (15.9, 26.4)
- added R8: 220, Resistor_THT:R_Axial_DIN0207_L6.3mm_D2.5mm_P10.16mm_Horizontal, F.Cu at (15.9, 30.4)
- added R9: 220, Resistor_THT:R_Axial_DIN0207_L6.3mm_D2.5mm_P10.16mm_Horizontal, F.Cu at (15.9, 34.5)
- added SW1: SW_Push, Button_Switch_THT:SW_PUSH_6mm, F.Cu at (29.7, 43.0)
- added SW2: SW_Push, Button_Switch_THT:SW_PUSH_6mm, F.Cu at (29.7, 51.6)
- added SW3: SW_Push, Button_Switch_THT:SW_PUSH_6mm, F.Cu at (29.7, 60.1)
- added SW4: SW_Nidec_CAS-120A1, Button_Switch_THT:SW_Slide_SPDT_Straight_CK_OS102011MS2Q, F.Cu at (68.0, 58.8)
- added U1: 4_Digits_7Seg_CC, New Library:4_Digits_7Seg, F.Cu at (97.8, 38.1)
- added U2: LD1117V33, Package_TO_SOT_THT:TO-220-3_Vertical, F.Cu at (67.3, 74.9)
- added U3: TP4056-42-ESOP8, Package_SO:SOIC-8-1EP_3.9x4.9mm_P1.27mm_EP2.41x3.3mm_ThermalVias, F.Cu at (31.9, 70.0)
- added U4: DW01A, Package_TO_SOT_SMD:SOT-23-6, F.Cu at (30.2, 75.6)
- added U5: EPM3064ATC100-7N, EPM3064:PLCC127P1765X1765X457-44N, F.Cu at (40.6, 27.3)
- added Y1: CXO_DIP8, Oscillator:Oscillator_DIP-8, F.Cu at (60.0, 52.0)

Commit message: Add files via upload
Parts:
- U1: value 4_Digits_7Seg_CC -> EPM3064ATC100-7N; footprint New Library:4_Digits_7Seg -> EPM3064:PLCC127P1765X1765X457-44N
- U3: value TP4056-42-ESOP8 -> 4_Digits_7Seg_CC; footprint Package_SO:SOIC-8-1EP_3.9x4.9mm_P1.27mm_EP2.41x3.3mm_ThermalVias -> New Library:4_Digits_7Seg
- U4: value DW01A -> TP4056-42-ESOP8; footprint Package_TO_SOT_SMD:SOT-23-6 -> Package_SO:SOIC-8-1EP_3.9x4.9mm_P1.27mm_EP2.41x3.3mm_ThermalVias
- U5: value EPM3064ATC100-7N -> DW01A; footprint EPM3064:PLCC127P1765X1765X457-44N -> Package_TO_SOT_SMD:SOT-23-6
- moved J3 182.9 mm to (230.5, 87.5)
- moved J1 173.1 mm to (223.1, 45.4)
- moved R3 170.3 mm to (230.3, 75.0)
- moved R4 170.3 mm to (230.3, 76.8)
- moved R5 170.3 mm to (230.3, 78.5)
- moved C5 170.3 mm to (227.9, 75.0)
- moved C6 170.3 mm to (227.9, 76.8)
- moved C1 168.5 mm to (225.4, 75.0)
- moved C2 168.5 mm to (225.4, 76.8)
- moved C3 168.5 mm to (225.4, 78.5)
- moved C4 168.5 mm to (225.4, 80.2)
- moved R1 168.5 mm to (227.9, 78.5)
- moved R2 168.5 mm to (227.9, 80.2)
- moved D1 159.2 mm to (231.5, 64.5)
- moved J2 156.7 mm to (197.2, 102.5), turned to 180 degrees
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Connections:
- C1 pad 1: VCC -> Vcc
- C2 pad 1: VCC -> Vcc
- C3 pad 1: VCC -> Vcc
- C4 pad 1: VCC -> Vcc
- C5 pad 1: VCC -> Vcc
- C6 pad 1: VCC -> Vcc
- C9 pad 1: Net-(U4-VCC) -> Net-(U5-VCC)
- J1 pad 4: VCC -> Vcc
- J2 pad 15: VCC -> Vcc
- J3 pad 1: VCC -> Vcc
- P1 pad A12: GND -> Net-(P1-GND-PadA1)
- P1 pad A5: Net-(D2-A) -> unconnected-(P1-CC-PadA5)
- P1 pad B12: GND -> Net-(P1-GND-PadA1)
- Q5 pad 4: Net-(U4-OD) -> Net-(U5-OD)
- Q5 pad 5: Net-(U4-OC) -> Net-(U5-OC)
- R10 pad 2: Net-(U1-e) -> Net-(U3-e)
- R11 pad 2: Net-(U1-f) -> Net-(U3-f)
- R12 pad 2: Net-(U1-g) -> Net-(U3-g)
- R13 pad 2: Net-(U1-DPX) -> Net-(U3-DPX)
- R2 pad 1: VCC -> Vcc
- R21 pad 2: Net-(U3-~{CHRG}) -> Net-(U4-~{CHRG})
- R22 pad 2: Net-(U3-~{STDBY}) -> Net-(U4-~{STDBY})
- R23 pad 2: Net-(U4-VCC) -> Net-(U5-VCC)
- R25 pad 1: Net-(U4-CS) -> Net-(U5-CS)
- R26 pad 1: Net-(U3-PROG) -> Net-(U4-PROG)
- R3 pad 1: VCC -> Vcc
- R4 pad 1: VCC -> Vcc
- R5 pad 1: VCC -> Vcc
- R6 pad 2: Net-(U1-a) -> Net-(U3-a)
- R7 pad 2: Net-(U1-b) -> Net-(U3-b)
- R8 pad 2: Net-(U1-c) -> Net-(U3-c)
- R9 pad 2: Net-(U1-d) -> Net-(U3-d)
- SW1 pad 1: VCC -> Vcc
- SW4 pad 1: GND -> OUT-
- SW4 pad 3: VCC -> Vcc
- U1 pad 1: Net-(U1-e) -> GCLKRn
- U1 pad 10: Net-(U1-f) -> GND
- U1 pad 11: Net-(U1-a) -> P11
- U1 pad 12: Net-(Q1-C) -> P12
- U1 pad 2: Net-(U1-d) -> GCLK2
- U1 pad 3: Net-(U1-DPX) -> Vcc
- U1 pad 4: Net-(U1-c) -> GND
- U1 pad 5: Net-(U1-g) -> GND
- U1 pad 6: Net-(Q4-C) -> GND
- U1 pad 7: Net-(U1-b) -> TDI
- U1 pad 8: Net-(Q3-C) -> P8
- U1 pad 9: Net-(Q2-C) -> P9
- U2 pad 3: Net-(BT1-+) -> unconnected-(U2-VI-Pad3)
- U3 pad 1: GND -> Net-(U3-e)
- U3 pad 2: Net-(U3-PROG) -> Net-(U3-d)
- U3 pad 3: GND -> Net-(U3-DPX)
- U3 pad 4: unconnected-(U3-V_{CC}-Pad4) -> Net-(U3-c)
- U3 pad 5: Net-(BT1-+) -> Net-(U3-g)
- U3 pad 6: Net-(U3-~{STDBY}) -> Net-(Q4-C)
- U3 pad 7: Net-(U3-~{CHRG}) -> Net-(U3-b)
- U3 pad 8: unconnected-(U3-CE-Pad8) -> Net-(Q3-C)
- U3 pad 9: unconnected-(U3-EPAD-Pad9) -> Net-(Q2-C)
- U4 pad 1: Net-(U4-OD) -> GND
- U4 pad 2: Net-(U4-CS) -> Net-(U4-PROG)
- U4 pad 3: Net-(U4-OC) -> GND
- U4 pad 5: Net-(U4-VCC) -> Net-(BT1-+)
- U4 pad 6: GND -> Net-(U4-~{STDBY})
- U5 pad 1: GCLKRn -> Net-(U5-OD)
- U5 pad 2: GCLK2 -> Net-(U5-CS)
- U5 pad 3: VCC -> Net-(U5-OC)
- U5 pad 4: GND -> unconnected-(U5-TD-Pad4)
- U5 pad 5: GND -> Net-(U5-VCC)
- Y1 pad 8: VCC -> Vcc
Routing:
- net Vcc: track 0.00 -> 18.1 mm
- net GCLK1: track 0.00 -> 11.8 mm
- net GND: track 0.00 -> 8.37 mm
