File: New_CPLD_Digtal_Clock_type-c_Battery/New_CPLD_Digtal_Clock_type-c_Battery.kicad_pcb (KiCad board)
At the start: 2 copper layers, 56 parts, among them J1 Conn_02x05_Odd_Even, J2 Conn_01x15, J3 Conn_01x15, P1 USB_C_Plug_USB2.0, Q1 CS9013, Q2 CS9013, Q3 CS9013, Q4 CS9013, Q5 FS8205A, SW1 SW_Push, SW2 SW_Push, SW3 SW_Push, SW4 SW_Nidec_CAS-120A1, U1 EPM3064ATC100-7N, U2 LD1117V33, U3 4_Digits_7Seg_CC, U4 TP4056-42-ESOP8, U5 DW01A, Y1 CXO_DIP8

Commit message: CPLD版本更新
Parts:
- removed Q5: FS8205A, FS8205A:SOP65P640X120-8N
- removed U1: EPM3064ATC100-7N, EPM3064:PLCC127P1765X1765X457-44N
- removed U3: 4_Digits_7Seg_CC, New Library:4_Digits_7Seg
- moved J3 102.3 mm to (138.4, 43.0)
- moved J1 96.4 mm to (126.7, 47.6)
- moved C1 90.2 mm to (141.3, 42.4)
- moved C2 90.2 mm to (141.3, 44.1)
- moved C3 90.2 mm to (141.3, 45.9)
- moved C4 90.2 mm to (141.3, 47.6)
- moved C5 90.2 mm to (143.7, 42.4)
- moved C6 90.2 mm to (143.7, 44.1)
- moved R1 90.2 mm to (143.7, 45.9)
- moved R2 90.2 mm to (143.7, 47.6)
- moved R3 90.2 mm to (146.2, 42.4)
- moved R4 90.2 mm to (146.2, 44.1)
- moved R5 90.2 mm to (146.2, 45.9)
- moved D1 89.7 mm to (142.8, 50.7)
- moved J2 86.1 mm to (135.1, 43.0), turned to 0 degrees
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Connections:
- net Vcc renamed VCC
- SW4 pad 1: OUT- -> GND
Routing:
- net VCC: track 18.1 -> 0.00 mm
- net GCLK1: track 11.8 -> 0.00 mm
- net GND: track 8.37 -> 0.00 mm
