File: Raspberry pi pico 2w/Raspberry pi pico 2w/SHIELDkicad_sch.kicad_sch (KiCad schematic)
At the start: 12 parts, among them M1005 4u7, M1006 4u7, M1007 4u7, M1008 4u7, M1009 4u7, M1010 4u7, M1011 4u7, U3 CYW43439KUBGT

Commit message: update
Parts:
- added C24, C28: 100n, symbol Device:C_Small
- added C29, C30: 4u7, symbol Device:C_Small
- added C31, C32: 10p, symbol Device:C_Small
- added C33, C34: 18p, symbol Device:C_Small
- added C35: NF, symbol Device:C_Small
- added C36: 0.3pF, symbol Device:C_Small
- added C37: 0.36pF, symbol Device:C_Small
- added FL1: LFB212G45CG7D227, LFB212G45CG7D227, symbol Raspberry pi pico 2w:LFB212G45CG7D227
- added Jumper: 0R, symbol Device:R_US
- added L4: 4n7, symbol Device:L
- added R21, R22, R23: 22R, symbol Device:R_US
- added Y2: 37.4MHz, symbol Device:Crystal
- C22: renamed from M1009; value 4u7 -> 1u; module M1005/X5R/20% -> M0603/X5R/20%
- L2: description M1608 -> (none)
- R20: value 200 -> 22R; Watt 63mW/1% -> 50mW/1%
- renumbered M1007 to C20, M1005 to C21, M1006 to C23, M1010 to C25, M1008 to C26, M1005 to C26, M1011 to C27
Connections:
- net GNDREF: now also C24.2, C28.2, C29.2, C30.2, C33.2, C34.1, C35.2, C37.2, FL1.2 (GND)
- net VDDC: now also C24.1
- net VIN_LDO: now also C22.1, U3.C7 (LDO_VDD1P5), U3.M2 (WLRF_VDD_1P35)
- net VOUT_3P3: now also C25.1, R20.2, U3.M1 (WLRF_PA_VDD)
- net at C27.2, U3.H1 (BT_PAVDD): now also R20.1, C29.1, C30.1; no longer R20.2
- net VDDBAT: now reaches U3.F6 (WCC_VDDIO)
- net VDDBAT: now also C28.1
- net WL_GPIO1: now reaches U3.H6 (GPIO_1)
- net at U3.H7 (SDIO_DATA_1): now also R22.2
- net at U3.J1 (WLRF_2G_ELG): now also L4.2
- net WL_GPIO2: now reaches U3.J6 (GPIO_0)
- net WL_CS: now reaches U3.J7 (SDIO_DATA_3)
- net at U3.K1 (WLRF_2G_RF): now also C31.1
- net at U3.K6 (SDIO_DATA_0): now also R23.2
- net WL_GPIO0: now reaches U3.L5 (GPIO_2)
- net WL_D: now reaches U3.L6 (SDIO_CMD)
- net WL_D: now also U3.L7 (SDIO_DATA_2), R22.1
- net at U3.M4 (WLRF_XTAL_XOP): now also C33.1, Y2.1
- net at U3.M5 (WLRF_XTAL_XON): now also R21.2
- net WL_CLK: now reaches U3.M7 (SDIO_CLK)
- net WL_CLK: now also R23.1
- new net: C34.2, R21.1, Y2.2
- new net: FL1.1 (IN), Jumper.2
- new net: C31.2, C32.1, FL1.3 (OUT)
- new net: C35.1, C36.1, Jumper.1
- new net: C36.2, C37.1
- new net: C32.2, L4.1
- no-connect marks 0 -> 9
Other:
- moved on the sheet: C21, C22, C23, C25, C26, C27, L3, R20
