File: Raspberry pi pico 2w/Raspberry pi pico 2w/Raspberry pi pico 2w.kicad_pcb (KiCad board)
At the start: 2 copper layers, 65 x 56 mm, 5 parts, among them J1 GPIO

Commit message: update
Parts:
- added C1: 100n, R_0402_1005Metric, F.Cu at (130.0, 58.0)
- added C10: 100n, R_0402_1005Metric, F.Cu at (130.0, 67.0)
- added C11: 100n, R_0402_1005Metric, F.Cu at (134.0, 58.0)
- added C12: 100n, R_0402_1005Metric, F.Cu at (134.0, 67.0)
- added C13: 100n, R_0402_1005Metric, F.Cu at (137.0, 58.0)
- added C14: 100n, R_0402_1005Metric, F.Cu at (137.0, 70.0)
- added C15: 100n, R_0402_1005Metric, F.Cu at (140.0, 58.0)
- added C16: 100n, R_0402_1005Metric, F.Cu at (140.0, 67.0)
- added C17: 100n, R_0402_1005Metric, F.Cu at (144.0, 58.0)
- added C18: 100n, R_0402_1005Metric, F.Cu at (144.0, 67.0)
- added C18: 15p, R_0402_1005Metric, F.Cu at (147.0, 57.0)
- added C19: 100n, R_0402_1005Metric, F.Cu at (148.0, 58.0)
- added C19: 15p, R_0402_1005Metric, F.Cu at (153.0, 57.0)
- added C20: 100n, R_0402_1005Metric, F.Cu at (128.0, 83.0)
- added C21: 100n, R_0402_1005Metric, F.Cu at (128.0, 86.0)
- added C22: 100n, R_0402_1005Metric, F.Cu at (128.0, 89.0)
- added C23: 100n, R_0402_1005Metric, F.Cu at (128.0, 92.0)
- added C24: 100n, R_0402_1005Metric, F.Cu at (128.0, 95.0)
- added C25: 100n, R_0402_1005Metric, F.Cu at (131.0, 83.0)
- added C26: 100n, R_0402_1005Metric, F.Cu at (131.0, 86.0)
- added C27: 100n, R_0402_1005Metric, F.Cu at (131.0, 89.0)
- added C28: 100n, R_0402_1005Metric, F.Cu at (131.0, 92.0)
- added C29: 100n, R_0402_1005Metric, F.Cu at (131.0, 95.0)
- added C30: 100n, R_0402_1005Metric, F.Cu at (135.0, 83.0)
- added C31: 100n, R_0402_1005Metric, F.Cu at (135.0, 86.0)
- added C32: 100n, R_0402_1005Metric, F.Cu at (135.0, 89.0)
- added C33: 100n, R_0402_1005Metric, F.Cu at (135.0, 95.0)
- added C34: 100n, R_0402_1005Metric, F.Cu at (138.0, 86.0)
- added C35: 100n, R_0402_1005Metric, F.Cu at (138.0, 89.0)
- added C36: 100n, R_0402_1005Metric, F.Cu at (138.0, 92.0)
- added C37: 100n, R_0402_1005Metric, F.Cu at (138.0, 95.0)
- added C4: 47u, C_0805_2012Metric, F.Cu at (121.0, 58.0)
- added C5: 47u, C_0805_2012Metric, F.Cu at (121.0, 70.0)
- added C6: 47u, C_0805_2012Metric, F.Cu at (125.0, 70.0)
- added C8: 100n, R_0402_1005Metric, F.Cu at (130.0, 61.0)
- added C9: 100n, R_0402_1005Metric, F.Cu at (130.0, 64.0)
- added D1: PMEG6010ELR, Diode_SMD:D_SOD-123W, F.Cu at (107.0, 60.0)
- added D2: Green, LED_SMD:LED_0603_1608Metric, F.Cu at (158.0, 52.0)
- added FL1: LFB212G45CG7D227, LFB212G45CG7D227, F.Cu at (127.0, 83.0)
- added IC1: RT6154AGQW, SON50P300X400X80-15N-D, F.Cu at (113.0, 64.0)
- added IC2: W25Q32RVXHJQ, SON50P300X200X40-9N, F.Cu at (150.0, 71.0)
- added J2: USB3_A, Connector_USB:USB_A_Molex_67643, F.Cu at (163.0, 65.0)
- added J3: Debug, Connector_PinHeader_2.54mm:PinHeader_1x03_P2.54mm_Vertical, F.Cu at (160.0, 55.0)
- added JP1: ID_WP, Jumper:SolderJumper-2_P1.3mm_Open_Pad1.0x1.5mm, F.Cu at (154.0, 50.0)
- added Jumper: 0R, Jumper:SolderJumper-2_P1.3mm_Open_Pad1.0x1.5mm, F.Cu at (127.0, 86.0)
- added L1: 4u7, C_0805_2012Metric, F.Cu at (121.0, 64.0)
- added L2: 2.2u, R_0402_1005Metric, F.Cu at (125.0, 89.0)
- added L3: 600R@100MHz, R_0402_1005Metric, F.Cu at (125.0, 92.0)
- added L4: 4n7, R_0402_1005Metric, F.Cu at (125.0, 95.0)
- added Q1: DMG1012T, Package_TO_SOT_SMD:SOT-523, F.Cu at (107.0, 55.0)
- added R1: 100k, R_0402_1005Metric, F.Cu at (108.0, 68.0)
- added R10: 4k7, R_0402_1005Metric, F.Cu at (155.0, 64.0)
- added R11: 10k, R_0402_1005Metric, F.Cu at (130.0, 73.0)
- added R12: 10k, R_0402_1005Metric, F.Cu at (132.0, 73.0)
- added R13: 10k, R_0402_1005Metric, F.Cu at (134.0, 73.0)
- added R14: 10k, R_0402_1005Metric, F.Cu at (136.0, 73.0)
- added R15: 10k, R_0402_1005Metric, F.Cu at (138.0, 73.0)
- added R16: 10k, R_0402_1005Metric, F.Cu at (140.0, 73.0)
- added R17: 10k, R_0402_1005Metric, F.Cu at (142.0, 73.0)
- added R18: 10k, R_0402_1005Metric, F.Cu at (144.0, 73.0)
- added R19: 10k, R_0402_1005Metric, F.Cu at (146.0, 73.0)
- added R2: 33k, R_0402_1005Metric, F.Cu at (108.0, 70.0)
- added R20: 22R, R_0402_1005Metric, F.Cu at (141.0, 83.0)
- added R21: 22R, R_0402_1005Metric, F.Cu at (141.0, 86.0)
- added R22: 22R, R_0402_1005Metric, F.Cu at (141.0, 89.0)
- added R23: 22R, R_0402_1005Metric, F.Cu at (141.0, 92.0)
- added R3: 100k, R_0402_1005Metric, F.Cu at (108.0, 72.0)
- added R4: 1k, R_0402_1005Metric, F.Cu at (155.0, 67.0)
- added R5: 1k, R_0402_1005Metric, F.Cu at (155.0, 70.0)
- added R6: 330R, R_0402_1005Metric, F.Cu at (158.0, 55.0)
- added R7: 4k7, R_0402_1005Metric, F.Cu at (152.0, 64.0)
- added R8: 4k7, R_0402_1005Metric, F.Cu at (152.0, 67.0)
- added R9: 4k7, R_0402_1005Metric, F.Cu at (155.0, 61.0)
- added U1: CAT24C256, Package_SO:SOIC-8_3.9x4.9mm_P1.27mm, F.Cu at (158.0, 64.0)
- added U2: RP2350A0A2, QFN-60-1EP_7x7mm_P0.4mm_EP3.4x3.4mm, F.Cu at (137.0, 64.0)
- added U3: CYW43439KUBGT, BGA63N40P7X12_287X487X55N, F.Cu at (133.0, 89.0)
- added Y1: 12MHz, Crystal_SMD_3225-4Pin_3.2x2.5mm, F.Cu at (150.0, 59.0)
- added Y2: 37.4MHz, Crystal_SMD_3225-4Pin_3.2x2.5mm, F.Cu at (143.0, 83.0)
Routing:
- net GND: track 0.00 -> 312.3 mm
- net +3V3: track 0.00 -> 267.4 mm
- net /ID_SDA: track 0.00 -> 75.5 mm
- net /ID_SCL: track 0.00 -> 72.9 mm
- net /GPIO2/SDA1: track 0.00 -> 61.9 mm
- net /GPIO3/SCL1: track 0.00 -> 59.7 mm
- net /GPIO26: track 0.00 -> 55.7 mm
- net /GPIO25: track 0.00 -> 52.8 mm
- net /GPIO24: track 0.00 -> 52.4 mm
- net /GPIO19/PCM.FS: track 0.00 -> 52.1 mm
- net /GPIO22: track 0.00 -> 50.7 mm
- net /GPIO21/PCM.DOUT: track 0.00 -> 50.4 mm
- net /GPIO23: track 0.00 -> 50.3 mm
- net /GPIO20/PCM.DIN: track 0.00 -> 50.0 mm
- net /GPIO17: track 0.00 -> 49.9 mm
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- added copper zone on B.Cu, net +3V3
- added copper zone on F.Cu, net +3V3
- added copper zone on In2.Cu, net +3V3
- added copper zone on F.Cu, net +5V
- added copper zone on B.Cu, net GND
- added copper zone on F.Cu, net GND
- added copper zone on In1.Cu, net GND
Other:
- copper layers 2 -> 4
