File: Raspberry pi pico 2w/Raspberry pi pico 2w/Raspberry pi pico 2w.kicad_sch (KiCad schematic)
At the start: 11 parts, among them J1 GPIO, U1 CAT24C256, U2 RP2350A

Commit message: update the ESP32 pcb layout
Parts:
- removed C2, C3: 100nF, symbol Device:C_Small
- removed U2: RP2350A, Package_DFN_QFN:QFN-60-1EP_7x7mm_P0.4mm_EP3.4x3.4mm, symbol MCU_RaspberryPi:RP2350A
- added C10, C17, C7, C8: 4u7, symbol Device:C_Small
- added C11, C12, C13, C14, C15, C16, C9: 100n, symbol Device:C_Small
- added C4, C5, C6: 47u, symbol Device:C_Small
- added D1: PMEG6010ELR, Diode_SMD:Nexperia_CFP3_SOD-123W, symbol Diode:PMEG6010ELR
- added IC1: RT6154AGQW, SON50P300X400X80-15N-D, symbol Raspberry pi pico 2w:RT6154AGQW
- added IC2: W25Q32RVXHJQ, SON50P300X200X40-9N, symbol Raspberry pi pico 2w:W25Q32RVXHJQ
- added J2: USB3_A, symbol Connector:USB3_A
- added L1: L, symbol Device:L
- added R10, R7, R8: 100K, symbol Device:R_US
- added R11: 1K, symbol Device:R_US
- added R12, R13: 200, symbol Device:R_US
- added R5: 5K6, symbol Device:R_US
- added R6: 10K, symbol Device:R_US
- added R9: 560K, symbol Device:R_US
- added U2: RP2350A0A2, Package_DFN_QFN:QFN-60-1EP_7x7mm_P0.4mm_EP3.4x3.4mm, symbol Raspberry pi pico 2w:RP2350A
Connections:
- net +1V1: now also C10.1, C14.1, C15.1, U2.23 (DVDD), U2.39 (DVDD), U2.6 (DVDD)
- net +3V3: now also C11.2, C12.2, C13.1, C16.1, C5.1, C6.1, C7.1, C8.1, C9.2, IC1.4 (VOUT_1), IC1.5 (VOUT_2), IC2.8 (VCC), R12.1, R9.1, U2.1 (IOVDD), U2.11 (IOVDD), U2.20 (IOVDD), U2.30 (IOVDD), U2.38 (IOVDD), U2.45 (IOVDD)
- net GNDREF: now also C10.2, C11.1, C12.1, C13.2, C14.2, C15.2, C16.2, C17.2, C4.2, C5.2, C6.2, C7.2, C8.2, C9.1, IC1.15 (PGND), IC2.4 (GND), J2.4 (GND), J2.8 (SSTX-), J2.9 (SSTX+), R10.2, R6.2, R8.2, U2.61 (GND)
- net GPIO0: now also U2.2 (GPIO0)
- net GPIO1: now also U2.3 (GPIO1)
- net GPIO10: now also U2.14 (GPIO10)
- net GPIO11: now also U2.15 (GPIO11)
- net GPIO12: now also U2.16 (GPIO12)
- net GPIO13: now also U2.17 (GPIO13)
- net GPIO14: now also U2.18 (GPIO14)
- net GPIO15: now also U2.19 (GPIO15)
- net GPIO16: now also U2.27 (GPIO16)
- net GPIO17: now also U2.28 (GPIO17)
- net GPIO18: now also U2.29 (GPIO18)
- net GPIO19: now also U2.31 (GPIO19)
- net GPIO2: now also U2.4 (GPIO2)
- net GPIO20: now also U2.32 (GPIO20)
- net GPIO21: now also U2.33 (GPIO21)
- net GPIO22: now also U2.34 (GPIO22)
- net GPIO23: now also U2.35 (GPIO23)
- net GPIO24: now also U2.36 (GPIO24)
- net GPIO25: now also U2.37 (GPIO25)
- net GPIO26/ADC01: now also U2.40 (GPIO26/ADC0)
- net GPIO27/ADC1: now also U2.41 (GPIO27/ADC1)
- net GPIO28/ADC2: now also U2.42 (GPIO28/ADC2)
- net GPIO29/ADC3: now also U2.43 (GPIO29/ADC3)
- net GPIO3: now also U2.5 (GPIO3)
- net GPIO4: now also U2.7 (GPIO4)
- net GPIO5: now also U2.8 (GPIO5)
- net GPIO6: now also U2.9 (GPIO6)
- net GPIO7: now also U2.10 (GPIO7)
- net GPIO8: now also U2.12 (GPIO8)
- net GPIO9: now also U2.13 (GPIO9)
- net QSPI_SCLK: now also IC2.6 (CLK), U2.56 (QSPI_SCLK)
- net QSPI_SD0: now also IC2.5 (DI_(IO0)), U2.57 (QSPI_SD0)
- net QSPI_SD1: now also IC2.2 (DO_(IO1)), U2.59 (QSPI_SD1)
- net QSPI_SD2: now also IC2.3 (~{WP_(IO2)}), U2.58 (QSPI_SD2)
- net QSPI_SD3: now also IC2.7 (~{HOLD_OR_}/RESET_(IO3)), U2.55 (QSPI_SD3)
- net QSPI_SS: now also IC2.1 (~{CS}), R11.2, U2.60 (~{QSPI_SS})
- net USB_DM: now also J2.2 (D-)
- net USB_DMX: now also U2.51 (USB_DM)
- net USB_DP: now also J2.3 (D+)
- net USB_DPX: now also U2.52 (USB_DP)
- net XIN: now also U2.21 (XIN)
- new net: C17.1, R13.1, U2.44 (ADC_AVDD)
- new net: IC1.3 (FB), R10.1, R9.2
- new net: IC1.6 (LX2_1), IC1.7 (LX2_2), L1.2
- new net: IC1.8 (LX1_1), IC1.9 (LX1_2), L1.1
- new net 3V3_EN: IC1.12 (EN), R7.2
- new net ADC_VREF: R12.2, R13.2
- new net RUN: U2.26 (RUN)
- new net SC: U2.24 (SWCLK)
- new net SD: U2.25 (SWDIO)
- new net TP4: IC1.13 (PS/SYNC), R8.1
- new net TP6: R11.1
- new net VBUS: D1.2 (A), J2.1 (VBUS), R5.1
- new net VSYS: C4.1, D1.1 (K), IC1.10 (VIN_1), IC1.11 (VIN_2), R7.1
- new net WL_GPIO2: R5.2, R6.1
- new net XOUT: U2.22 (XOUT)
- no-connect marks 3 -> 5
Other:
- moved on the sheet: J1, R3, R4

Commit message: update
Parts:
- added C18, C19: 15p, symbol Device:C_Small
- added D2: Green, symbol Device:D
- added J3: Conn_01x03, symbol Connector_Generic:Conn_01x03
- added R14: 1K, symbol Device:R_US
- added R15, R16, R17: 470, symbol Device:R_US
- added Y1: Crystal, symbol Device:Crystal
- R5: description M0603 -> (none)
Connections:
- net GNDREF: now also C18.2, C19.2, D2.1 (K)
- net XIN: now also C18.1, Y1.1
- net XOUT: now also R14.2
- new net: C19.1, R14.1, Y1.2
- new net TP0: D2.2 (A), R15.1
- new net WL_GPIO0: R15.2

Commit message: update
Parts:
- added Q1: DMG1012T, Package_TO_SOT_SMD:SOT-523, symbol Transistor_FET:DMG1012T
- added R18: 20K, symbol Device:R_US
- added R19: 10K, symbol Device:R_US
- R16, R17: value 470 -> 100
Connections:
- net GNDREF: now also J3.2 (Pin_2), R19.1
- net SC: now also R16.2
- net SD: now also R17.2
- net VSYS: now also R18.2
- net SWCLK: now reaches J3.1 (Pin_1)
- net SWCLK: now also R16.1
- net SWDIO: now reaches J3.3 (Pin_3)
- net SWDIO: now also R17.1
- new net: Q1.3 (D), R18.1
- new net WL_CLK: Q1.2 (S), R19.2
- new net WL_CS: Q1.1 (G)
Other:
- added sheet SHIELD (SHIELDkicad_sch.kicad_sch)
- moved on the sheet: J3

Commit message: update
Other:
- added sheet EXPANSION (Expansion.kicad_sch)
Changed lines of the file:
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@@
+		)
+	)
+	(sheet
+		(at 92.19 216.61)
+		(size 69.85 54.61)
+		(exclude_from_sim no)
+		(in_bom yes)
+		(on_board yes)
+		(dnp no)
+		(fields_autoplaced yes)
+		(stroke
+			(width 0.1524)
+			(type solid)
+		)
+		(fill
+			(color 0 0 0 0)
+		)
+		(property "Sheetname" "EXPANSION"
+			(at 92.19 216.4584 0)
+			(show_name no)
+			(do_not_autoplace no)
+			(effects
+				(font
+					(size 1.27 1.27)
+				)
+				(justify left bottom)
+			)
+		)
+		(property "Sheetfile" "Expansion.kicad_sch"
+			(at 92.19 271.0946 0)
+			(show_name no)
+			(do_not_autoplace no)
+			(effects
+				(font
+					(size 1.27 1.27)
+				)
+				(justify left top)
+			)
+		)
+		(instances
+			(project "Raspberry pi pico 2w"
+				(path "/e63e39d7-6ac0-4ffd-8aa3-1841a4541b55"
+					(page "3")
+				)
+			)
 		)
 	)
