File: ESP32-S3-DevKitC-1_V1.1/ESP32-S3-DevKitC-1_V1.1.kicad_pcb (KiCad board)
At the start: 2 copper layers, 46 parts, among them J2 Conn_01x22, J3 Conn_01x22, P1 USB_C_Plug_USB2.0, P2 USB_C_Plug_USB2.0, Q3 L8050QLT1G, Q4 L8050QLT1G, SW1 NTC013-AT1J-A160T, SW2 NTC013-AT1J-A160T, U1 CP2102N-Axx-xQFN28, U4 ESP32-S3-WROOM-1

Commit message: New update
Parts:
- added C9: 0.1uF, Capacitor_SMD:C_0603_1608Metric, F.Cu at (125.0, 87.3)
- added R14: 0, Resistor_SMD:R_0603_1608Metric, F.Cu at (133.0, 94.8)
- added R15: 0, Resistor_SMD:R_0603_1608Metric, F.Cu at (133.0, 97.3)
- moved U4 58.5 mm to (143.5, 72.0), turned to 0 degrees
- moved R7 47.8 mm to (129.0, 97.3)
- moved R6 42.2 mm to (129.0, 94.8)
- moved R10 37.8 mm to (129.0, 104.8)
- moved P2 36.7 mm to (142.1, 100.0), turned to 0 degrees
- moved R9 35.7 mm to (129.0, 102.3), turned to 0 degrees
- moved P1 35.5 mm to (142.1, 90.7), turned to 0 degrees
- moved R12 29.2 mm to (133.0, 89.8)
- moved R13 29.2 mm to (133.0, 92.3)
- moved R8 27.6 mm to (129.0, 99.8)
- moved R11 26.0 mm to (133.0, 87.3), turned to 0 degrees
- moved R4 25.3 mm to (129.0, 89.8)
- moved Q3 20.9 mm to (161.0, 95.2), turned to 0 degrees
- moved SW2 18.3 mm to (152.9, 92.6)
- moved U1 17.8 mm to (160.0, 89.6)
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
Commit message: update the ESP32 pcb layout
Parts:
- added IC1: SGM2212-3.3XKC3G_TR, ESP32-S3-DevKitC-1_V1.1:SOT230P700X180-4N, F.Cu at (132.2, 109.3)
- added SW3: SW_Push, Button_Switch_SMD:SW_SPST_Omron_B3FS-100xP, F.Cu at (109.0, 70.5)
- added SW4: SW_Push, Button_Switch_SMD:SW_SPST_Omron_B3FS-100xP, F.Cu at (104.0, 110.5)
- J3: value Conn_01x22 -> Conn01x02
- moved R12 75.7 mm to (207.7, 102.5)
- moved U4 71.6 mm to (213.1, 89.0), turned to -90 degrees
- moved C3 71.3 mm to (192.0, 85.6), turned to 90 degrees
- moved R15 68.1 mm to (201.0, 102.2), turned to 180 degrees
- moved C7 64.0 mm to (183.8, 90.0), turned to 90 degrees
- moved R2 63.5 mm to (186.6, 89.3)
- moved R3 62.7 mm to (191.5, 82.5), turned to 180 degrees
- moved R4 60.7 mm to (189.7, 91.2)
- moved D9 57.5 mm to (102.5, 80.1), turned to 180 degrees
- moved C20 56.1 mm to (180.8, 93.5), turned to 180 degrees
- moved C15 55.8 mm to (180.8, 96.0), turned to 180 degrees
- moved D12 55.3 mm to (106.3, 79.6), turned to -90 degrees
- moved D6 54.1 mm to (216.5, 103.2), turned to 180 degrees
- moved R7 53.7 mm to (181.2, 84.8), turned to 180 degrees
- moved R5 52.0 mm to (180.8, 98.0)
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Routing:
- net Net-(R15-Pad2): track 0.00 -> 283.9 mm
- net GNDREF: track 0.00 -> 277.3 mm, vias 0 -> 1
- net /GPIO0: track 0.00 -> 210.5 mm
- net +3V3: track 0.00 -> 136.2 mm
- net +5V: track 0.00 -> 111.1 mm, vias 0 -> 2
- net /USB_DP: track 0.00 -> 108.7 mm
- net /U0RXD: track 0.00 -> 84.5 mm
- net /U0TXD: track 0.00 -> 59.0 mm
- net /CHIP_PU: track 0.00 -> 48.8 mm
- net VBUS: track 0.00 -> 33.4 mm
- net Net-(U1-VBUS): track 0.00 -> 19.6 mm, vias 0 -> 2
- net Net-(Q3-C): track 0.00 -> 12.4 mm
- net Net-(C9-Pad2): track 0.00 -> 11.8 mm
- net Net-(Q4-B): track 0.00 -> 11.2 mm
- net Net-(Q3-B): track 0.00 -> 10.7 mm
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
Commit message: update
Routing:
- net +5V: track 111.1 -> 107.9 mm
- net GNDREF: track 277.3 -> 279.1 mm
Changed lines of the file:
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@@
 		(start 181.92979 78)
 		(end 179.0968 80.83299)
-		(width 0.2032)
-		(layer "F.Cu")
-		(net "GNDREF")
-	)
-	(segment
-		(start 127.917 105.918)
-		(end 129.032 107.033)
-		(width 0.2032)
+		(width 0.5)
 		(layer "F.Cu")
 		(net "GNDREF")
@@
 		(start 211.31 87.5)
 		(end 213.25 87.5)
-		(width 0.2032)
+		(width 0.5)
 		(layer "F.Cu")
 		(net "GNDREF")
@@
 	)
 	(segment
+		(start 123.685 105.815)
+		(end 124.5 105)
+		(width 0.5)
+		(layer "F.Cu")
+		(net "GNDREF")
+	)
+	(segment
 		(start 218.33 102.295)
 		(end 218.25 102.375)
@@
 	)
 	(segment
+		(start 123.685 111.76)
+		(end 123.685 107.188)
+		(width 0.5)
+		(layer "F.Cu")
+		(net "GNDREF")
+	)
+	(segment
 		(start 106.299 80.289)
 		(end 105.9494 80.6386)
@@
 	)
 	(segment
+		(start 129.032 105.532)
+		(end 129.032 107.033)
+		(width 0.5)
+		(layer "F.Cu")
+		(net "GNDREF")
+	)
+	(segment
 		(start 95.7825 72.5)
 		(end 97.5 72.5)
@@
 	)
 	(segment
-		(start 123.685 107.188)
-		(end 123.685 106.058)
-		(width 0.2032)
-		(layer "F.Cu")
-		(net "GNDREF")
-	)
-	(segment
-		(start 123.685 107.188)
-		(end 123.685 111.76)
-		(width 0.2032)
+		(start 124.5 105)
+		(end 128.5 105)
+		(width 0.5)
 		(layer "F.Cu")
 		(net "GNDREF")
@@
 		(start 194.8662 75.1338)
 		(end 192 78)
-		(width 0.2032)
+		(width 0.5)
 		(layer "F.Cu")
 		(net "GNDREF")
@@
 		(start 182.235048 89.0266)
 		(end 186.438648 84.823)
-		(width 0.2032)
+		(width 0.5)
 		(layer "F.Cu")
 		(net "GNDREF")
@@
 		(start 219.329 81.421)
 		(end 219.329 77.216)
-		(width 0.2032)
+		(width 0.5)
 		(layer "F.Cu")
 		(net "GNDREF")
@@
 	)
 	(segment
+		(start 128.5 105)
+		(end 129.032 105.532)
+		(width 0.5)
+		(layer "F.Cu")
+		(net "GNDREF")
+	)
+	(segment
 		(start 116.84 96.139)
 		(end 116.84 96.876)
@@
 		(start 219.329 77.216)
 		(end 217.2468 75.1338)
-		(width 0.2032)
+		(width 0.5)
 		(layer "F.Cu")
 		(net "GNDREF")
@@
 	)
 	(segment
-		(start 123.825 105.918)
-		(end 127.917 105.918)
-		(width 0.2032)
-		(layer "F.Cu")
-		(net "GNDREF")
-	)
-	(segment
 		(start 183.769 88.773)
 		(end 183.769 89.268)
@@
 		(start 217.2468 75.1338)
 		(end 194.8662 75.1338)
-		(width 0.2032)
+		(width 0.5)
 		(layer "F.Cu")
 		(net "GNDREF")
@@
 		(start 179.0968 80.83299)
 		(end 179.0968 88.111712)
-		(width 0.2032)
+		(width 0.5)
 		(layer "F.Cu")
 		(net "GNDREF")
@@
 		(start 218.33 81.2032)
 		(end 212.0332 87.5)
-		(width 0.2032)
+		(width 0.5)
 		(layer "F.Cu")
 		(net "GNDREF")
@@
 	)
 	(segment
+		(start 123.685 107.188)
+		(end 123.685 105.815)
+		(width 0.5)
+		(layer "F.Cu")
+		(net "GNDREF")
+	)
+	(segment
 		(start 98.975 101.775)
 		(end 99 101.75)
@@
 	)
 	(segment
-		(start 123.685 106.058)
-		(end 123.825 105.918)
-		(width 0.2032)
-		(layer "F.Cu")
-		(net "GNDREF")
-	)
-	(segment
 		(start 104.975 68.225)
 		(end 105 68.25)
@@
 		(start 180.011688 89.0266)
 		(end 182.235048 89.0266)
-		(width 0.2032)
+		(width 0.5)
 		(layer "F.Cu")
 		(net "GNDREF")
@@
 		(start 179.0968 88.111712)
 		(end 180.011688 89.0266)
-		(width 0.2032)
+		(width 0.5)
 		(layer "F.Cu")
 		(net "GNDREF")
@@
 		(start 192 78)
 		(end 181.92979 78)
-		(width 0.2032)
+		(width 0.5)
 		(layer "F.Cu")
 		(net "GNDREF")
@@
 		(start 213.25 87.5)
 		(end 219.329 81.421)
-		(width 0.2032)
+		(width 0.5)
 		(layer "F.Cu")
 		(net "GNDREF")
@@
 		(start 218.33 97.75)
 		(end 218.33 102.295)
-		(width 0.2032)
+		(width 0.5)
 		(layer "F.Cu")
 		(net "GNDREF")
@@
 		(start 163.021106 119.9286)
 		(end 186.5 96.449706)
-		(width 0.2032)
+		(width 0.5)
 		(layer "F.Cu")
 		(net "/USB_DP")
@@
 		(start 133.236 107.237)
 		(end 135.332 109.333)
-		(width 0.2032)
+		(width 0.5)
 		(layer "F.Cu")
 		(net "+3V3")
@@
 		(start 192.024 91.821)
 		(end 190.246 93.599)
-		(width 0.2032)
+		(width 0.5)
 		(layer "F.Cu")
 		(net "+3V3")
@@
 		(start 131.14 109.333)
 		(end 129.032 109.333)
-		(width 0.2032)
+		(width 0.5)
 		(layer "F.Cu")
 		(net "+3V3")
@@
 		(start 192.75 82.5)
 		(end 193.5 83.25)
-		(width 0.2032)
+		(width 0.5)
 		(layer "F.Cu")
 		(net "+3V3")
@@
 		(start 187.4642 93.599)
 		(end 187.4642 94.0948)
-		(width 0.2032)
+		(width 0.5)
 		(layer "F.Cu")
 		(net "+3V3")
@@
 		(start 193.373 86.373)
 		(end 192.024 86.373)
-		(width 0.2032)
+		(width 0.5)
 		(layer "F.Cu")
 		(net "+3V3")
@@
 		(start 193.5 83.25)
 		(end 193.5 86.246)
-		(width 0.2032)
+		(width 0.5)
 		(layer "F.Cu")
 		(net "+3V3")
@@
 		(start 151.848 109.333)
 		(end 161.387 118.872)
-		(width 0.2032)
+		(width 0.5)
 		(layer "F.Cu")
 		(net "+3V3")
@@
 		(start 135.332 109.333)
 		(end 151.848 109.333)
-		(width 0.2032)
+		(width 0.5)
 		(layer "F.Cu")
 		(net "+3V3")
@@
 		(start 133.236 107.237)
 		(end 131.14 109.333)
-		(width 0.2032)
+		(width 0.5)
 		(layer "F.Cu")
 		(net "+3V3")
@@
 		(start 190.246 93.599)
 		(end 187.4642 93.599)
-		(width 0.2032)
+		(width 0.5)
 		(layer "F.Cu")
 		(net "+3V3")
@@
 		(start 187.4642 89.3064)
 		(end 187.4642 93.599)
-		(width 0.2032)
+		(width 0.5)
 		(layer "F.Cu")
 		(net "+3V3")
@@
 		(start 133.236 103.505)
 		(end 133.236 107.237)
-		(width 0.2032)
+		(width 0.5)
 		(layer "F.Cu")
 		(net "+3V3")
@@
 		(start 192.024 86.373)
 		(end 192.024 91.821)
-		(width 0.2032)
+		(width 0.5)
 		(layer "F.Cu")
 		(net "+3V3")
@@
 		(start 187.4642 94.0948)
 		(end 162.687 118.872)
-		(width 0.2032)
+		(width 0.5)
 		(layer "F.Cu")
 		(net "+3V3")
@@
 	)
 	(segment
-		(start 125.235 114.985)
-		(end 125.235 111.76)
-		(width 0.2032)
-		(layer "F.Cu")
-		(net "+5V")
-	)
-	(segment
 		(start 117.67979 62.81925)
 		(end 122.17884 58.3202)
@@
 		(start 129.032 111.633)
 		(end 125.362 111.633)
-		(width 0.2032)
+		(width 0.5)
 		(layer "F.Cu")
 		(net "+5V")
@@
 		(start 125.235 107.188)
 		(end 125.235 111.76)
-		(width 0.2032)
+		(width 0.5)
 		(layer "F.Cu")
 		(net "+5V")
@@
 		(layer "F.Cu")
 		(net "+5V")
-	)
-	(segment
-		(start 125.25 115)
-		(end 125.235 114.985)
-		(width 0.2032)
-		(layer "F.Cu")
-		(net "+5V")

Commit message: update
Changed lines of the file:
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@@
 		(start 104.975 62.75)
 		(end 104.975 68.225)
-		(width 0.2032)
+		(width 0.5)
 		(layer "F.Cu")
 		(net "GNDREF")
@@
 		(start 106.299 80.289)
 		(end 105.9494 80.6386)
-		(width 0.2032)
+		(width 0.5)
 		(layer "F.Cu")
 		(net "GNDREF")
@@
 		(start 111 68.25)
 		(end 111 75)
-		(width 0.2032)
+		(width 0.5)
 		(layer "F.Cu")
 		(net "GNDREF")
@@
 		(start 113.538 96.851)
 		(end 110.134 96.851)
-		(width 0.2032)
+		(width 0.5)
 		(layer "F.Cu")
 		(net "GNDREF")
@@
 		(start 95.7825 72.5)
 		(end 97.5 72.5)
-		(width 0.2032)
+		(width 0.5)
 		(layer "F.Cu")
 		(net "GNDREF")
@@
 		(start 116.84 96.876)
 		(end 118.126 96.876)
-		(width 0.2032)
+		(width 0.5)
 		(layer "F.Cu")
 		(net "GNDREF")
@@
 		(start 116.84 96.876)
 		(end 113.563 96.876)
-		(width 0.2032)
+		(width 0.5)
 		(layer "F.Cu")
 		(net "GNDREF")
@@
 		(start 118.25 97)
 		(end 118.25 110.286)
-		(width 0.2032)
+		(width 0.5)
 		(layer "F.Cu")
 		(net "GNDREF")
@@
 		(start 159.85 57)
 		(end 122.25 57)
-		(width 0.2032)
+		(width 0.5)
 		(layer "F.Cu")
 		(net "GNDREF")
@@
 		(start 102.3306 80.6386)
 		(end 101.829 80.137)
-		(width 0.2032)
+		(width 0.5)
 		(layer "F.Cu")
 		(net "GNDREF")
@@
 		(start 110.109 96.876)
 		(end 106.705 96.876)
-		(width 0.2032)
+		(width 0.5)
 		(layer "F.Cu")
 		(net "GNDREF")
@@
 		(start 129.032 106.159)
 		(end 131.686 103.505)
-		(width 0.2032)
+		(width 0.5)
 		(layer "F.Cu")
 		(net "GNDREF")
@@
 		(start 97.9195 80.137)
 		(end 95.7825 78)
-		(width 0.2032)
+		(width 0.5)
 		(layer "F.Cu")
 		(net "GNDREF")
@@
 		(start 105.9494 80.6386)
 		(end 102.3306 80.6386)
-		(width 0.2032)
+		(width 0.5)
 		(layer "F.Cu")
 		(net "GNDREF")
@@
 		(start 117 77)
 		(end 117 75)
-		(width 0.2032)
+		(width 0.5)
 		(layer "F.Cu")
 		(net "GNDREF")
@@
 		(start 97.5 72.5)
 		(end 101.75 68.25)
-		(width 0.2032)
+		(width 0.5)
 		(layer "F.Cu")
 		(net "GNDREF")
@@
 		(start 113 68.25)
 		(end 111 68.25)
-		(width 0.2032)
+		(width 0.5)
 		(layer "F.Cu")
 		(net "GNDREF")
@@
 		(start 119.761 93.218)
 		(end 116.84 96.139)
-		(width 0.2032)
+		(width 0.5)
 		(layer "F.Cu")
 		(net "GNDREF")
@@
 		(start 131.686 101.219)
 		(end 131.686 103.505)
-		(width 0.2032)
+		(width 0.5)
 		(layer "F.Cu")
 		(net "GNDREF")
@@
 		(start 101.829 80.137)
 		(end 97.9195 80.137)
-		(width 0.2032)
+		(width 0.5)
 		(layer "F.Cu")
 		(net "GNDREF")
@@
 		(start 106.299 80.289)
 		(end 113.711 80.289)
-		(width 0.2032)
+		(width 0.5)
 		(layer "F.Cu")
 		(net "GNDREF")
@@
 		(start 113.711 80.289)
 		(end 117 77)
-		(width 0.2032)
+		(width 0.5)
 		(layer "F.Cu")
 		(net "GNDREF")
@@
 		(start 117 75)
 		(end 111 75)
-		(width 0.2032)
+		(width 0.5)
 		(layer "F.Cu")
 		(net "GNDREF")
@@
 		(start 101.75 68.25)
 		(end 105 68.25)
-		(width 0.2032)
+		(width 0.5)
 		(layer "F.Cu")
 		(net "GNDREF")
@@
 		(start 112.975 64.75)
 		(end 112.975 68.225)
-		(width 0.2032)
+		(width 0.5)
 		(layer "F.Cu")
 		(net "GNDREF")
@@
 		(start 118.25 110.286)
 		(end 117.404 111.132)
-		(width 0.2032)
+		(width 0.5)
 		(layer "F.Cu")
 		(net "GNDREF")
@@
 		(start 131.6505 98.552)
 		(end 131.6505 101.1835)
-		(width 0.2032)
+		(width 0.5)
 		(layer "F.Cu")
 		(net "GNDREF")
@@
 		(start 122.225 59.5)
 		(end 122.225 64.375)
-		(width 0.2032)
+		(width 0.5)
 		(layer "F.Cu")
 		(net "GNDREF")
@@
 		(start 122.25 57)
 		(end 122.25 59.5)
-		(width 0.2032)
+		(width 0.5)
 		(layer "B.Cu")
 		(net "GNDREF")
@@
 		(start 116.7774 98.2586)
 		(end 116.7774 112.6242)
-		(width 0.2032)
+		(width 0.5)
 		(layer "F.Cu")
 		(net "/USB_DP")
@@
 		(start 134.316 100.139)
 		(end 133.236 101.219)
-		(width 0.2032)
+		(width 0.5)
 		(layer "F.Cu")
 		(net "+3V3")
@@
 		(start 133.236 101.219)
 		(end 133.236 103.505)
-		(width 0.2032)
+		(width 0.5)
 		(layer "F.Cu")
 		(net "+3V3")
@@
 		(start 136.398 100.139)
 		(end 137.605 100.139)
-		(width 0.2032)
+		(width 0.5)
 		(layer "F.Cu")
 		(net "+3V3")
@@
 		(start 123.698 88.265)
 		(end 123.698 90.17)
-		(width 0.2032)
+		(width 0.5)
 		(layer "F.Cu")
 		(net "+3V3")
@@
 		(start 138.049 99.695)
 		(end 138.049 96.774)
-		(width 0.2032)
+		(width 0.5)
 		(layer "F.Cu")
 		(net "+3V3")
@@
 		(start 121.92 88.202)
 		(end 123.635 88.202)
-		(width 0.2032)
+		(width 0.5)
 		(layer "F.Cu")
 		(net "+3V3")
@@
 		(start 137.605 100.139)
 		(end 138.049 99.695)
-		(width 0.2032)
+		(width 0.5)
 		(layer "F.Cu")
 		(net "+3V3")
@@
 		(start 122.8054 91.0626)
 		(end 123.698 90.17)
-		(width 0.2032)
+		(width 0.5)
 		(layer "F.Cu")
 		(net "+3V3")
@@
 		(start 122.8054 94.3574)
 		(end 122.8054 91.0626)
-		(width 0.2032)
+		(width 0.5)
 		(layer "F.Cu")
 		(net "+3V3")
@@
 		(start 125.222 96.774)
 		(end 122.8054 94.3574)
-		(width 0.2032)
+		(width 0.5)
 		(layer "F.Cu")
 		(net "+3V3")
@@
 		(start 136.398 100.139)
 		(end 134.316 100.139)
-		(width 0.2032)
+		(width 0.5)
 		(layer "F.Cu")
 		(net "+3V3")
@@
 		(start 138.049 96.774)
 		(end 125.222 96.774)
-		(width 0.2032)
+		(width 0.5)
 		(layer "F.Cu")
 		(net "+3V3")
@@
 		(start 106.68 98.171)
 		(end 106.1784 97.6694)
-		(width 0.2032)
+		(width 0.5)
 		(layer "F.Cu")
 		(net "VBUS")
@@
 		(start 109.5378 92.95)
 		(end 114.25 92.95)
-		(width 0.2032)
+		(width 0.5)
 		(layer "F.Cu")
 		(net "VBUS")
@@
 		(start 106.299 78.969)
 		(end 106.299 76.77)
-		(width 0.2032)
+		(width 0.5)
 		(layer "F.Cu")
 		(net "VBUS")
@@
 		(start 106.299 76.77)
 		(end 98 76.77)
-		(width 0.2032)
+		(width 0.5)
 		(layer "F.Cu")
 		(net "VBUS")
@@
 		(start 106.299 76.77)
 		(end 115.303 76.77)
-		(width 0.2032)
+		(width 0.5)
 		(layer "F.Cu")
 		(net "VBUS")
@@
 		(start 106.1784 96.3094)
 		(end 109.5378 92.95)
-		(width 0.2032)
+		(width 0.5)
 		(layer "F.Cu")
 		(net "VBUS")
@@
 		(start 98 76.77)
 		(end 95.7825 76.77)
-		(width 0.2032)
+		(width 0.5)
 		(layer "F.Cu")
 		(net "VBUS")
@@
 		(start 106.1784 97.6694)
 		(end 106.1784 96.3094)
-		(width 0.2032)
+		(width 0.5)
 		(layer "F.Cu")
 		(net "VBUS")
@@
 		(start 117.67979 62.81925)
 		(end 122.17884 58.3202)
-		(width 0.2032)
+		(width 0.5)
 		(layer "F.Cu")
 		(net "+5V")
@@
 		(start 117.090421 89.55)
 		(end 114.25 89.55)
-		(width 0.2032)
+		(width 0.5)
 		(layer "F.Cu")
 		(net "+5V")
@@
 		(start 115.316 73.357)
 		(end 116.893 73.357)
-		(width 0.2032)
+		(width 0.5)
 		(layer "F.Cu")
 		(net "+5V")
@@
 		(start 117.67979 72.57021)
 		(end 117.67979 62.81925)
-		(width 0.2032)
+		(width 0.5)
 		(layer "F.Cu")
 		(net "+5V")
@@
 		(start 122.17884 58.3202)
 		(end 134.460621 58.3202)
-		(width 0.2032)
+		(width 0.5)
 		(layer "F.Cu")
 		(net "+5V")
@@
 		(start 136.6748 60.53438)
 		(end 136.6748 69.965621)
-		(width 0.2032)
+		(width 0.5)
 		(layer "F.Cu")
 		(net "+5V")
@@
 		(start 116.893 73.357)
 		(end 117.67979 72.57021)
-		(width 0.2032)
+		(width 0.5)
 		(layer "F.Cu")
 		(net "+5V")
@@
 		(start 136.6748 69.965621)
 		(end 117.090421 89.55)
-		(width 0.2032)
+		(width 0.5)
 		(layer "F.Cu")
 		(net "+5V")
@@
 		(start 134.460621 58.3202)
 		(end 136.6748 60.53438)
-		(width 0.2032)
+		(width 0.5)
 		(layer "F.Cu")
 		(net "+5V")
@@
 		(start 106.525 62.75)
 		(end 117.61054 62.75)
-		(width 0.2032)
-		(layer "F.Cu")
-		(net "+5V")
+		(width 0.5)
+		(layer "F.Cu")
+		(net "+5V")

Commit message: update
Connections:
- U1 pad : (no net) -> GNDREF
- U4 pad : (no net) -> GNDREF
Routing:
- net GNDREF: track 279.1 -> 434.3 mm, vias 1 -> 3
- net VBUS: track 33.4 -> 170.7 mm, vias 0 -> 2
- net /GPIO20: track 0.00 -> 109.7 mm, vias 0 -> 2
- net +3V3: track 136.2 -> 242.0 mm, vias 0 -> 4
- net /CHIP_PU: track 48.8 -> 152.3 mm, vias 0 -> 2
- net /GPIO19: track 0.06 -> 100.1 mm, vias 0 -> 2
- net /USB_DN: track 0.00 -> 84.3 mm, vias 0 -> 2
- net +5V: track 107.9 -> 189.3 mm, vias 2 -> 4
- net /USB_DP: track 108.7 -> 189.3 mm, vias 0 -> 2
- net /RTS: track 5.87 -> 67.3 mm
- net /DTR: track 5.13 -> 54.9 mm
- net /U0TXD: track 59.0 -> 106.1 mm, vias 0 -> 2
- net Net-(Q4-E): track 0.00 -> 15.7 mm
- net VCC: track 0.00 -> 8.00 mm
- net Net-(R15-Pad2): track 283.9 -> 291.9 mm
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- added copper zone on B.Cu, net GNDREF
- added copper zone on F.Cu, net GNDREF
Other:
- board outline added: 155 x 73 mm
