File: Raspberry pi 5/ComputeModule4.kicad_sch (KiCad schematic)
At the start: 13 parts, among them J2 USB4105-GF-A, J3 SM04B-SRSS-TB

Commit message: update the ComputeModule4
Parts:
- added J4: DNP, symbol Connector_Generic:Conn_01x10
- added JP2: SolderJumper_2_Open, symbol Jumper:SolderJumper_2_Open
- J3: value SM04B-SRSS-TB -> SM04B-SRSS-TB(LF)(SN)
Connections:
- net GND: now also U3.1 (GND), U3.14 (GND), U3.2 (GND), U3.22 (GND), U3.23 (GND), U3.32 (GND), U3.33 (GND), U3.42 (GND), U3.43 (GND), U3.52 (GND), U3.53 (GND), U3.59 (GND), U3.60 (GND), U3.65 (GND), U3.66 (GND), U3.7 (GND), U3.71 (GND), U3.74 (GND), U3.8 (GND), J4.2 (Pin_2), JP2.2 (B)
- net nLED_Activity: now also U3.21 (PI_nLED_Activity)
- net nPWR_LED: now also U3.95 (nPI_LED_PWR)
- net EEPROM_nWP: now reaches U3.20 (EEPROM_nWP)
- net EEPROM_nWP: now also JP2.1 (A)
- net GPIO07: now reaches U3.37 (GPIO07)
- net GPIO07: now also J4.9 (Pin_9)
- net GPIO11: now reaches U3.38 (GPIO11)
- net GPIO11: now also J4.7 (Pin_7)
- net GPIO08: now reaches U3.39 (GPIO08)
- net GPIO08: now also J4.8 (Pin_8)
- net GPIO09: now reaches U3.40 (GPIO09)
- net GPIO09: now also J4.6 (Pin_6)
- net GPIO10: now reaches U3.44 (GPIO10)
- net GPIO10: now also J4.5 (Pin_5)
- net GPIO15: now reaches U3.51 (GPIO15)
- net GPIO15: now also J4.4 (Pin_4)
- net GPIO14: now reaches U3.55 (GPIO14)
- net GPIO14: now also J4.3 (Pin_3)
- net GPIO03: now reaches U3.56 (GPIO03)
- net GPIO02: now reaches U3.58 (GPIO02)
- net 3.3V: now reaches U3.78 (GPIO_VREF(1.8v/3.3v_Input))
- net 3.3V: now also U3.84 (+3.3v_(Output)), U3.86 (+3.3v_(Output))
- net 5V: now reaches U3.79 (+5v_(Input))
- net 5V: now also U3.81 (+5v_(Input)), U3.83 (+5v_(Input)), U3.85 (+5v_(Input)), U3.87 (+5v_(Input))
- net 1.8V: now reaches U3.88 (+1.8v_(Output))
- net 1.8V: now also U3.90 (+1.8v_(Output))
- net nRPIBOOT: now reaches U3.93 (nRPIBOOT)
- net nRPIBOOT: now also J4.10 (Pin_10)
- new net 3v3: J4.1 (Pin_1)
Other:
- note added: "1"
- note added: "2"
- note added: "Activity LED"
- note added: "Close for EEPROM write protection"
- note added: "GPIO"
- note added: "PWR LED"
- note added: "Qwiic/Stemma"
- note added: "SPIO_CE0"
- note added: "SPIO_CE1"
- note added: "SPIO_CLK"
- note added: "SPIO_MISO"
- note added: "SPIO_MOSI"
- note added: "UART_RXD"
- note added: "UART_TXD"
- note added: "USB-C (Power Only)"
- note added: "nBOOT"
- title: (none) -> Raspberry Pi Compute Module 4 Base Carrier
- moved on the sheet: J3, R7, R8

Commit message: add CM4 Ethernet and High Speed
Parts:
- renumbered U3 to Module1A
Changed lines of the file:
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@@
 		(dnp no)
 		(fields_autoplaced yes)
-		(property "Reference" "U3"
+		(property "Reference" "Module1A"
 			(at 74.93 43.18 0)
 			(show_name no)
@@
 			(project "Raspberry pi 5"
 				(path "/e63e39d7-6ac0-4ffd-8aa3-1841a4541b55/c93c5551-bbc2-499a-9f11-7ebb9b21275e"
-					(reference "U3")
+					(reference "Module1A")
 					(unit 1)
 				)

Commit message: update the Ethernet IO Board
Parts:
- removed Module1A: (no value), symbol 2x DF40C-100D5-0.4V:2x_DF40C-100D5-0.4V
- added U11: (no value), symbol 2x DF40C-100DS-0.4V:Module1A
Connections:
- net 1.8V: now also U11.88 (+1.8v_(Output)), U11.90 (+1.8v_(Output))
- net 3.3V: now also U11.78 (GPIO_VREF(1.8v/3.3v_Input)), U11.84 (+3.3v_(Output)), U11.86 (+3.3v_(Output))
- net 5V: now also U11.79 (+5v_(Input)), U11.81 (+5v_(Input)), U11.83 (+5v_(Input)), U11.85 (+5v_(Input)), U11.87 (+5v_(Input))
- net EEPROM_nWP: now also U11.20 (EEPROM_nWP)
- net GND: now also U11.1 (GND), U11.14 (GND), U11.2 (GND), U11.22 (GND), U11.23 (GND), U11.32 (GND), U11.33 (GND), U11.42 (GND), U11.43 (GND), U11.52 (GND), U11.53 (GND), U11.59 (GND), U11.60 (GND), U11.65 (GND), U11.66 (GND), U11.7 (GND), U11.71 (GND), U11.74 (GND), U11.8 (GND), U11.98 (GND)
- net GPIO02: now also U11.58 (GPIO02)
- net GPIO03: now also U11.56 (GPIO03)
- net GPIO07: now also U11.37 (GPIO07)
- net GPIO08: now also U11.39 (GPIO08)
- net GPIO09: now also U11.40 (GPIO09)
- net GPIO10: now also U11.44 (GPIO10)
- net GPIO11: now also U11.38 (GPIO11)
- net GPIO14: now also U11.55 (GPIO14)
- net GPIO15: now also U11.51 (GPIO15)
- net nLED_Activity: now also U11.21 (PI_nLED_Activity)
- net nPWR_LED: now also U11.95 (nPI_LED_PWR)
- net nRPIBOOT: now also U11.93 (nRPIBOOT)
