File: Raspberry pi 5/CM4 PCIe.kicad_sch (KiCad schematic)
At the start: 0 parts

Commit message: update the cm4 USB port
Parts:
- added C10, C5, C6, C7, C8, C9: 10u 35v, symbol Device:C
- added C11, C4: 100n, symbol Device:C
- added C12, C14: nf, symbol Device:C
- added C13: 1.2nF, symbol Device:C
- added C15, C16, C17, C18: 10u, symbol Device:C
- added C19: 100uF, symbol Device:C
- added J13: 10018783-11200TLF, 10018783-11200TLF:AMPHENOL_10018783-11200TLF, symbol 10018783-11200TLF:10018783-11200TLF
- added L1: SRN6045TA-3R3Y, SRN6045TA330M, symbol SRN6045TA-3R3Y:SRN6045TA-3R3Y
- added R20: 10R, symbol Device:R_US
- added R21, R22: 12k 1%, symbol Device:R_US
- added R23: 15k 1%, symbol Device:R_US
- added TP3: TestPoint, symbol Connector:TestPoint
- added U12: AP64501SP-13, AP64501SP-13:SOIC127P600X170-9N, symbol AP64501SP-13:AP64501SP-13
Connections:
- new net: C13.1, R21.1
- new net: C4.2, U12.1 (BST)
- new net: C11.1, U12.4 (SS)
- new net: C12.1, C14.2, R21.2, R22.1, R23.2, U12.5 (FB), U12.6 (COMP)
- new net: L1.1, R20.2, U12.8 (SW)
- new net: C4.1, R20.1
- new net +12v: C10.1, C5.1, C6.1, C7.1, C8.1, C9.1, J13.A2 (+12v), J13.A3 (+12v), J13.B1 (+12v), J13.B2 (+12v), J13.B3 (+12v), U12.2 (VIN), U12.3 (EN)
- new net +3.3V: J13.A10 (+3.3v), J13.A5 (TCK), J13.A6 (TDI), J13.A8 (TMS), J13.A9 (+3.3v), J13.B10 (+3.3vAUX), J13.B8 (+3.3v), J13.B9 (nTRST)
- new net +3.3v: C14.1, C15.1, C16.1, C17.1, C18.1, C19.1, L1.2, R22.2, TP3.1
- new net GNDREF: C10.2, C11.2, C12.2, C13.2, C15.2, C16.2, C17.2, C18.2, C19.2, C5.2, C6.2, C7.2, C8.2, C9.2, J13.A12 (GND), J13.A15 (GND), J13.A18 (GND), J13.A4 (GND), J13.A7 (TD0), J13.B13 (GND), J13.B16 (GND), J13.B18 (GND), J13.B4 (GND), R23.1, U12.7 (GND), U12.9 (EP)
- new net PCIE_CLK_N: J13.A14 (REFCLK-)
- new net PCIE_CLK_P: J13.A13 (REFCLK+)
- new net PCIE_CLK_nREQ: J13.B12 (nCLKREQ)
- new net PCIE_CRX_N: J13.A16 (PREP0)
- new net PCIE_RX_P: J13.A17 (PREN0)
- new net PCIE_TX_N: J13.B14 (PETP0)
- new net PCIE_TX_P: J13.B15 (PETN0)
- new net PCIE_nRST: J13.A11 (nPERST)
- no-connect marks 0 -> 6
Other:
- note added: "NB PCIe x1 tasks a maximum of +12v @0.6A or +3.3v @3A, 10Watts combined TX and RX have PN swaps to improve routing"
- title: (none) -> Compute Module 4 IO Board - PCIe
