File: Raspberry pi 5/CM4 USB.kicad_sch (KiCad schematic)
At the start: 0 parts

Commit message: update the cm4 USB port
Parts:
- added C20, C21, C22: C, symbol Device:C
- added C23, C24, C25, C26: 10u, symbol Device:C
- added C27: 100uF, symbol Device:C
- added IC1: AP22653W6, SOT95P280X145-6N, symbol AP22653W6-7:AP22653W6-7
- added J20: USB_OTG, symbol Connector:USB_OTG
- added J21: Conn_02x05_Odd_Even, symbol Connector_Generic:Conn_02x05_Odd_Even
- added R24: 2.2k 1%, symbol Device:R_US
- added R25: 12k 1%, symbol Device:R_US
- added R26, R27, R28, R29: 36k 1%, symbol Device:R_US
- added R30: R_US, symbol Device:R_US
- added U13: USB2514B_Bi, Package_DFN_QFN:QFN-36-1EP_6x6mm_P0.5mm_EP3.7x3.7mm, symbol Interface_USB:USB2514B_Bi
- added U14: FSUSB42MUX, Package_SO:MSOP-10_3x3mm_P0.5mm, symbol Interface_USB:FSUSB42MUX
- added U15: TPD4EUSB30, Package_SON:USON-10_2.5x1.0mm_P0.5mm, symbol Power_Protection:TPD4EUSB30
- added Y1: 24MHz, symbol Device:Crystal
Connections:
- new net: IC1.5 (ILIM), R30.1
- new net: C23.1, C24.1, C25.1, C26.1, C27.1, IC1.6 (OUT)
- new net: R25.2, U13.35 (RBIAS)
- new net: C20.1, U13.33 (XTALIN/CLKIN), Y1.1
- new net: R28.1, U13.28 (SUSP_IND/LOCAL_PWR/NON_REM0)
- new net: C21.1, U13.32 (XTALOUT), Y1.2
- new net: R27.1, U13.22 (SDA/SMBDATA/NON_REM1)
- new net: R26.1, U13.24 (SCL/SMBCLK/CFG_SEL0)
- new net: R29.1, U13.25 (HS_IND/CFG_SEL1)
- new net +3.3v: U13.10 (VDDA33), U13.15 (VDD33), U13.23 (VDD33), U13.27 (VBUS_DET), U13.29 (VDDA33), U13.36 (VDDA33), U13.5 (VDDA33), U14.1 (VCC)
- new net +5v: C22.1, IC1.1 (IN)
- new net GNDREF: C20.2, C21.2, C22.2, C23.2, C24.2, C25.2, C26.2, C27.2, IC1.2 (GND), J20.5 (GND), J20.SH (Shield), J21.7 (Pin_7), J21.8 (Pin_8), R24.2, R25.1, R26.2, R27.2, R28.2, R29.2, R30.2, U13.37 (VSS), U14.10 (~{OE}), U14.5 (GND), U15.3 (GND), U15.8 (GND)
- new net HD1_N: U13.1 (USBDM_DN1/PRT_DIS_M1)
- new net HD1_P: U13.2 (USBDP_DN1/PRT_DIS_P1)
- new net HD2_N: U13.3 (USBDM_DN2/PRT_DIS_M2)
- new net HD2_P: U13.4 (USBDP_DN2/PRT_DIS_P2)
- new net HD3_N: J21.3 (Pin_3), U13.6 (USBDM_DN3/PRT_DIS_M3)
- new net HD3_P: J21.5 (Pin_5), U13.7 (USBDP_DN3/PRT_DIS_P3)
- new net HD4_N: J21.4 (Pin_4), U13.8 (USBDM_DN4/PRT_DIS_M4)
- new net HD4_P: J21.6 (Pin_6), U13.9 (USBDP_DN4/PRT_DIS_P4)
- new net PWR: IC1.3 (EN)
- new net PWR1: U13.12 (PRTPWR1/BC_EN1)
- new net USB2_N: U14.4 (D-)
- new net USB2_P: U14.3 (D+)
- new net USBD_N: J20.2 (D-), U14.8 (HSD2-), U15.4 (D2+)
- new net USBD_P: J20.3 (D+), U14.9 (HSD2+), U15.5 (D2-)
- new net USBH_N: U13.30 (USBDM_UP), U14.6 (HSD1-)
- new net USBH_P: U13.31 (USBDP_UP), U14.7 (HSD1+)
- new net USBOTG: J20.1 (VBUS), R24.1, U14.2 (SEL)
- new net VBUS: J21.1 (Pin_1), J21.2 (Pin_2)
- new net nEXTRST: U13.26 (RESET_N)
- new net nOCS1: IC1.4 (~{FAULT}), U13.13 (OCS_N1), U13.17 (OCS_N2), U13.19 (OCS_N3), U13.21 (OCS_N4)
- no-connect marks 0 -> 6
Other:
- note added: "Current Limit switch"
- note added: "Expansion USB connector"
- note added: "If a cable in plugged into the USB socket the CM4 becomes a usb device"
- note added: "Stacked USB connectors"
- note added: "USB 2.0 Hub"
- title: (none) -> Compute Module 4 IO Board - USB
