File: Raspberry pi 5/Raspberry pi 5.kicad_sch (KiCad schematic)
At the start: 6 parts, among them J1 GPIO, U1 CAT24C256

Commit message: Update the CM4 RTC Fan, PSUs, and Motherboard
Other:
- added sheet CM4 PSUs (CM4 PSUs.kicad_sch)
- added sheet CM4 RTC Fan (CM4 RTC Fan.kicad_sch)
- added sheet Motherboard (Motherboard.kicad_sch)
Changed lines of the file:
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@@
 	)
 	(sheet
-		(at 163.83 49.53)
+		(at 162.56 99.06)
+		(size 43.18 31.75)
+		(exclude_from_sim no)
+		(in_bom yes)
+		(on_board yes)
+		(dnp no)
+		(fields_autoplaced yes)
+		(stroke
+			(width 0.1524)
+			(type solid)
+		)
+		(fill
+			(color 0 0 0 0)
+		)
+		(property "Sheetname" "CM4 RTC Fan"
+			(at 162.56 98.3484 0)
+			(show_name no)
+			(do_not_autoplace no)
+			(effects
+				(font
+					(size 1.27 1.27)
+				)
+				(justify left bottom)
+			)
+		)
+		(property "Sheetfile" "CM4 RTC Fan.kicad_sch"
+			(at 162.56 131.3946 0)
+			(show_name no)
+			(do_not_autoplace no)
+			(effects
+				(font
+					(size 1.27 1.27)
+				)
+				(justify left top)
+			)
+		)
+		(instances
+			(project "Raspberry pi 5"
+				(path "/e63e39d7-6ac0-4ffd-8aa3-1841a4541b55"
+					(page "7")
+				)
+			)
+		)
+	)
+	(sheet
+		(at 118.11 139.7)
+		(size 40.64 27.94)
+		(exclude_from_sim no)
+		(in_bom yes)
+		(on_board yes)
+		(dnp no)
+		(fields_autoplaced yes)
+		(stroke
+			(width 0.1524)
+			(type solid)
+		)
+		(fill
+			(color 0 0 0 0)
+		)
+		(property "Sheetname" "CM4 PSUs"
+			(at 118.11 138.9884 0)
+			(show_name no)
+			(do_not_autoplace no)
+			(effects
+				(font
+					(size 1.27 1.27)
+				)
+				(justify left bottom)
+			)
+		)
+		(property "Sheetfile" "CM4 PSUs.kicad_sch"
+			(at 118.11 168.2246 0)
+			(show_name no)
+			(do_not_autoplace no)
+			(effects
+				(font
+					(size 1.27 1.27)
+				)
+				(justify left top)
+			)
+		)
+		(instances
+			(project "Raspberry pi 5"
+				(path "/e63e39d7-6ac0-4ffd-8aa3-1841a4541b55"
+					(page "8")
+				)
+			)
+		)
+	)
+	(sheet
+		(at 162.56 17.78)
 		(size 43.18 29.21)
 		(exclude_from_sim no)
@@
 		)
 		(property "Sheetname" "CM4 High Speed"
-			(at 163.83 48.8184 0)
+			(at 162.56 17.0684 0)
 			(show_name no)
 			(do_not_autoplace no)
@@
 		)
 		(property "Sheetfile" "CM4 High Speed.kicad_sch"
-			(at 163.83 79.3246 0)
+			(at 162.56 47.5746 0)
 			(show_name no)
 			(do_not_autoplace no)
@@
 	)
 	(sheet
-		(at 162.56 88.9)
+		(at 161.29 57.15)
 		(size 43.18 33.02)
 		(exclude_from_sim no)
@@
 		)
 		(property "Sheetname" "CM4 PCIe"
-			(at 162.56 88.1884 0)
+			(at 161.29 56.4384 0)
 			(show_name no)
 			(do_not_autoplace no)
@@
 		)
 		(property "Sheetfile" "CM4 PCIe.kicad_sch"
-			(at 162.56 122.5046 0)
+			(at 161.29 90.7546 0)
 			(show_name no)
 			(do_not_autoplace no)
@@
 	)
 	(sheet
-		(at 118.11 88.9)
+		(at 116.84 57.15)
 		(size 41.91 33.02)
 		(exclude_from_sim no)
@@
 		)
 		(property "Sheetname" "CM4 Ethernet"
-			(at 118.11 88.1884 0)
+			(at 116.84 56.4384 0)
 			(show_name no)
 			(do_not_autoplace no)
@@
 		)
 		(property "Sheetfile" "CM4 Ethernet.kicad_sch"
-			(at 118.11 122.5046 0)
+			(at 116.84 90.7546 0)
 			(show_name no)
 			(do_not_autoplace no)
@@
 	)
 	(sheet
-		(at 118.11 49.53)
+		(at 116.84 17.78)
 		(size 43.18 30.48)
 		(exclude_from_sim no)
@@
 		)
 		(property "Sheetname" "ComputeModule4"
-			(at 118.11 48.8184 0)
+			(at 116.84 17.0684 0)
 			(show_name no)
 			(do_not_autoplace no)
@@
 		)
 		(property "Sheetfile" "ComputeModule4.kicad_sch"
-			(at 118.11 80.5946 0)
+			(at 116.84 48.8446 0)
 			(show_name no)
 			(do_not_autoplace no)
@@
 	)
 	(sheet
-		(at 119.38 130.81)
+		(at 118.11 99.06)
 		(size 40.64 31.75)
 		(exclude_from_sim no)
@@
 		)
 		(property "Sheetname" "CM4 USB"
-			(at 119.38 130.0984 0)
+			(at 118.11 98.3484 0)
 			(show_name no)
 			(do_not_autoplace no)
@@
 		)
 		(property "Sheetfile" "CM4 USB.kicad_sch"
-			(at 119.38 163.1446 0)
+			(at 118.11 131.3946 0)
 			(show_name no)
 			(do_not_autoplace no)
@@
 				)
 			)
+		)
+	)
+	(sheet
+		(at 162.56 139.7)
+		(size 41.91 26.67)
+		(exclude_from_sim no)
+		(in_bom yes)
+		(on_board yes)
+		(dnp no)
+		(fields_autoplaced yes)
+		(stroke
+			(width 0.1524)
+			(type solid)
+		)
+		(fill
+			(color 0 0 0 0)
+		)
+		(property "Sheetname" "Motherboard"
+			(at 162.56 138.9884 0)
+			(show_name no)
+			(do_not_autoplace no)
+			(effects
+				(font
+					(size 1.27 1.27)
+				)
+				(justify left bottom)
+			)
+		)
+		(property "Sheetfile" "Motherboard.kicad_sch"
+			(at 162.56 166.9546 0)
+			(show_name no)
+			(do_not_autoplace no)
+			(effects
+				(font
+					(size 1.27 1.27)
+				)
+				(justify left top)
+			)
+		)
+		(instances
+			(project "Raspberry pi 5"
+				(path "/e63e39d7-6ac0-4ffd-8aa3-1841a4541b55"
+					(page "9")
+				)
+			)
