File: Windows_Hello_Camera/Windows_Hello_Camera.kicad_sch (KiCad schematic)
At the start: 2 parts, among them J1 Analog, J2 Digital

Commit message: mini 小鋼琴電子電路
Other:
- added sheet Power_Supply (Power_Supply.kicad_sch)
